Commit message: Ajustes e Organização do Pacote de Simulação do Robô - Integração URDF, Rviz e Gazebo

File: work_ws/dev_ws/src/salamander_bot/description/colors.xacro (robot description, xacro)
@@ -2,14 +2,17 @@
 <robot xmlns:xacro="http://www.ros.org/wiki/xacro">
     <material name="white">
-        <color rgba="1 1 1 1"/>
+        <color rgba="1.0 1.0 1.0 1.0"/>
     </material>
     <material name="orange">
-        <color rgba="1 0.3 0.1 1"/>
+        <color rgba="1.0 0.3 0.1 1.0"/>
     </material>
     <material name="blue">
-        <color rgba="0.2 0.2 1 1"/>
+        <color rgba="0.2 0.2 1.0 1.0"/>
     </material>
     <material name="black">
-        <color rgba="0 0 0 1"/>
+        <color rgba="0.0 0.0 0.0 1.0"/>
+    </material>
+    <material name="silver">
+        <color rgba="0.7 0.7 0.7 1.0"/>
     </material>
 </robot>

File: work_ws/dev_ws/src/salamander_bot/description/robot.urdf.xacro (robot description, xacro)
@@ -1,4 +1,4 @@
 <?xml version="1.0"?>
-<robot xmlns:xacro="http://www.ros.org/wiki/xacro"  name="robot">
+<robot name="salamander_bot" xmlns:xacro="http://www.ros.org/wiki/xacro">
     <!-- Robot Core File -->
     <xacro:include filename="robot_core.xacro" />

File: work_ws/dev_ws/src/salamander_bot/description/robot_core.xacro (robot description, xacro)
@@ -1,50 +1,161 @@
-<?xml version="1.0"?>
+<?xml version="1.0" ?>
 <robot xmlns:xacro="http://www.ros.org/wiki/xacro">
-    <xacro:include filename="colors.xacro" />
-    <link name="base_link"></link>
-    <!-- CHASSIS -->
-    <joint name="chassis_joint" type="fixed">
-        <parent link="base_link"/>
-        <child link="chassis"/>
-        <origin xyz="-0.1 0 0"/>
-    </joint>
-    <link name="chassis">
-        <visual>
-            <origin xyz="0.15 0 0.075" rpy="0 0 0"/>
-            <geometry>
-                <box size="0.43 0.25 0.15"/>
-            </geometry>
-            <material name="white"/>
-        </visual>
-    </link>
-        <!-- LEFT WHEEL -->
-    <joint name="left_wheel_joint" type="continuous">
-        <parent link="base_link"/>
-        <child link="left_wheel"/>
-        <origin xyz="0 0.05675 0" rpy="-${pi/2} 0 0"/>
-        <axis xyz="0 0 4"/>
-    </joint>
-    <link name="left_wheel">
-        <visual>
-            <geometry>
-                <cylinder length="0.04" radius="0.05" />
-            </geometry>
-            <material name="blue"/>
-        </visual>
-    </link>
-    <!-- RIGHT WHEEL -->
-    <joint name="right_wheel_joint" type="continuous">
-        <parent link="base_link"/>
-        <child link="right_wheel"/>
-        <origin xyz="0 -0.05675 0" rpy="${pi/2} 0 0"/>
-        <axis xyz="0 0 -1"/>
-    </joint>
-    <link name="right_wheel">
-        <visual>
-            <geometry>
-                <cylinder length="0.04" radius="0.05" />
-            </geometry>
-            <material name="blue"/>
-        </visual>
-    </link>
+<xacro:include filename="$(find salamander_bot)/description/colors.xacro" />
+<xacro:include filename="$(find salamander_bot)/description/salamander_bot.ros2control" />
+<xacro:include filename="$(find salamander_bot)/description/salamander_bot.gazebo" />
+<link name="base_link"></link>
+<link name="chassis">
+  <inertial>
+    <origin xyz="-0.031027251343893784 0.006588573186617724 0.08110908537527221" rpy="0 0 0"/>
+    <mass value="4.3632165889636445"/>
+    <inertia ixx="0.042227" iyy="0.075384" izz="0.090994" ixy="0.004338" iyz="-0.000531" ixz="0.008602"/>
+  </inertial>
+  <visual>
+    <origin xyz="0 0 0" rpy="0 0 0"/>
+    <geometry>
+      <mesh filename="file://$(find salamander_bot)/meshes/base_link.stl" scale="0.001 0.001 0.001"/>
+    </geometry>
+    <material name="silver"/>
+  </visual>
+  <collision>
+    <origin xyz="0 0 0" rpy="0 0 0"/>
+    <geometry>
+      <mesh filename="file://$(find salamander_bot)/meshes/base_link.stl" scale="0.001 0.001 0.001"/>
+    </geometry>
+  </collision>
+</link>
+<link name="wheel_lf_1">
+  <inertial>
+    <origin xyz="6.732011406662686e-09 0.013415334217220576 -2.2496351934075953e-09" rpy="0 0 0"/>
+    <mass value="0.2163222450067834"/>
+    <inertia ixx="8.8e-05" iyy="0.00011" izz="8.8e-05" ixy="0.0" iyz="-0.0" ixz="0.0"/>
+  </inertial>
+  <visual>
+    <origin xyz="-0.11315 -0.142 -0.03865" rpy="0 0 0"/>
+    <geometry>
+      <mesh filename="file://$(find salamander_bot)/meshes/wheel_lf_1.stl" scale="0.001 0.001 0.001"/>
+    </geometry>
+    <material name="black"/>
+  </visual>
+  <collision>
+    <origin xyz="-0.11315 -0.142 -0.03865" rpy="0 0 0"/>
+    <geometry>
+      <mesh filename="file://$(find salamander_bot)/meshes/wheel_lf_1.stl" scale="0.001 0.001 0.001"/>
+    </geometry>
+  </collision>
+</link>
+<link name="wheel_lb_1">
+  <inertial>
+    <origin xyz="3.7014641768307044e-09 0.01344735270580652 -3.504848446189701e-09" rpy="0 0 0"/>
+    <mass value="0.21632224500656735"/>
+    <inertia ixx="8.8e-05" iyy="0.00011" izz="8.8e-05" ixy="-0.0" iyz="-0.0" ixz="0.0"/>
+  </inertial>
+  <visual>
+    <origin xyz="0.11315 -0.142 -0.03865" rpy="0 0 0"/>
+    <geometry>
+      <mesh filename="file://$(find salamander_bot)/meshes/wheel_lb_1.stl" scale="0.001 0.001 0.001"/>
+    </geometry>
+    <material name="black"/>
+  </visual>
+  <collision>
+    <origin xyz="0.11315 -0.142 -0.03865" rpy="0 0 0"/>
+    <geometry>
+      <mesh filename="file://$(find salamander_bot)/meshes/wheel_lb_1.stl" scale="0.001 0.001 0.001"/>
+    </geometry>
+  </collision>
+</link>
+<link name="wheel_rf_1">
+  <inertial>
+    <origin xyz="6.7541714166008404e-09 -0.013367918230393266 -2.072007607156756e-09" rpy="0 0 0"/>
+    <mass value="0.21632224116980406"/>
+    <inertia ixx="8.8e-05" iyy="0.00011" izz="8.8e-05" ixy="-0.0" iyz="0.0" ixz="0.0"/>
+  </inertial>
+  <visual>
+    <origin xyz="-0.11315 0.142 -0.03865" rpy="0 0 0"/>
+    <geometry>
+      <mesh filename="file://$(find salamander_bot)/meshes/wheel_rf_1.stl" scale="0.001 0.001 0.001"/>
+    </geometry>
+    <material name="black"/>
+  </visual>
+  <collision>
+    <origin xyz="-0.11315 0.142 -0.03865" rpy="0 0 0"/>
+    <geometry>
+      <mesh filename="file://$(find salamander_bot)/meshes/wheel_rf_1.stl" scale="0.001 0.001 0.001"/>
+    </geometry>
+  </collision>
+</link>
+<link name="wheel_rb_1">
+  <inertial>
+    <origin xyz="3.723448854797695e-09 -0.013447353552784869 -3.327369837990979e-09" rpy="0 0 0"/>
+    <mass value="0.21632224116958718"/>
+    <inertia ixx="8.8e-05" iyy="0.00011" izz="8.8e-05" ixy="0.0" iyz="0.0" ixz="0.0"/>
+  </inertial>
+  <visual>
+    <origin xyz="0.11315 0.142 -0.03865" rpy="0 0 0"/>
+    <geometry>
+      <mesh filename="file://$(find salamander_bot)/meshes/wheel_rb_1.stl" scale="0.001 0.001 0.001"/>
+    </geometry>
+    <material name="black"/>
+  </visual>
+  <collision>
+    <origin xyz="0.11315 0.142 -0.03865" rpy="0 0 0"/>
+    <geometry>
+      <mesh filename="file://$(find salamander_bot)/meshes/wheel_rb_1.stl" scale="0.001 0.001 0.001"/>
+    </geometry>
+  </collision>
+</link>
+<link name="rplidar_a1m8_1">
+  <inertial>
+    <origin xyz="0.0008205477062011579 0.0006535114455110541 0.017493457828168968" rpy="0 0 0"/>
+    <mass value="0.036021408390687064"/>
+    <inertia ixx="1.5e-05" iyy="1.2e-05" izz="2.3e-05" ixy="0.0" iyz="-0.0" ixz="-0.0"/>
+  </inertial>
+  <visual>
+    <origin xyz="0.077204 0.064205 -0.2095" rpy="0 0 0"/>
+    <geometry>
+      <mesh filename="file://$(find salamander_bot)/meshes/rplidar_a1m8_1.stl" scale="0.001 0.001 0.001"/>
+    </geometry>
+    <material name="blue"/>
+  </visual>
+  <collision>
+    <origin xyz="0.077204 0.064205 -0.2095" rpy="0 0 0"/>
+    <geometry>
+      <mesh filename="file://$(find salamander_bot)/meshes/rplidar_a1m8_1.stl" scale="0.001 0.001 0.001"/>
+    </geometry>
+  </collision>
+</link>
+<joint name="chassis_joint" type="fixed">
+  <parent link="base_link"/>
+  <child link="chassis"/>
+  <origin xyz="0.0 0.0 0.0"/>
+</joint>
+<joint name="wheel_lf_joint" type="continuous">
+  <origin xyz="0.11315 0.142 0.03865" rpy="0 0 0"/>
+  <parent link="base_link"/>
+  <child link="wheel_lf_1"/>
+  <axis xyz="0.0 1.0 0.0"/>
+</joint>
+<joint name="wheel_lb_joint" type="continuous">
+  <origin xyz="-0.11315 0.142 0.03865" rpy="0 0 0"/>
+  <parent link="base_link"/>
+  <child link="wheel_lb_1"/>
+  <axis xyz="0.0 1.0 0.0"/>
+</joint>
+<joint name="wheel_rf_joint" type="continuous">
+  <origin xyz="0.11315 -0.142 0.03865" rpy="0 0 0"/>
+  <parent link="base_link"/>
+  <child link="wheel_rf_1"/>
+  <axis xyz="0.0 1.0 0.0"/>
+</joint>
+<joint name="wheel_rb_joint" type="continuous">
+  <origin xyz="-0.11315 -0.142 0.03865" rpy="0 0 0"/>
+  <parent link="base_link"/>
+  <child link="wheel_rb_1"/>
+  <axis xyz="0.0 1.0 0.0"/>
+</joint>
+<joint name="rplidar_a1m8_joint" type="fixed">
+  <origin xyz="-0.077204 -0.064205 0.2095" rpy="0 0 0"/>
+  <parent link="base_link"/>
+  <child link="rplidar_a1m8_1"/>
+</joint>
 </robot>
