Commit message: leitura

File: work_ws/src/salamander_bot/description/robot_core.xacro (robot description, xacro)
@@ -105,24 +105,4 @@
   </collision>
 </link>
-<link name="rplidar_a1m8_1">
-  <inertial>
-    <origin xyz="0.0008205477062011579 0.0006535114455110541 0.017493457828168968" rpy="0 0 0"/>
-    <mass value="0.036021408390687064"/>
-    <inertia ixx="1.5e-05" iyy="1.2e-05" izz="2.3e-05" ixy="0.0" iyz="-0.0" ixz="-0.0"/>
-  </inertial>
-  <visual>
-    <origin xyz="0.077204 0.064205 -0.2095" rpy="0 0 0"/>
-    <geometry>
-      <mesh filename="file://$(find salamander_bot)/meshes/rplidar_a1m8_1.stl" scale="0.001 0.001 0.001"/>
-    </geometry>
-    <material name="blue"/>
-  </visual>
-  <collision>
-    <origin xyz="0.077204 0.064205 -0.2095" rpy="0 0 0"/>
-    <geometry>
-      <mesh filename="file://$(find salamander_bot)/meshes/rplidar_a1m8_1.stl" scale="0.001 0.001 0.001"/>
-    </geometry>
-  </collision>
-</link>
 <joint name="chassis_joint" type="fixed">
   <parent link="base_link"/>
@@ -154,8 +134,3 @@
   <axis xyz="0.0 1.0 0.0"/>
 </joint>
-<joint name="rplidar_a1m8_joint" type="fixed">
-  <origin xyz="-0.077204 -0.064205 0.2095" rpy="0 0 0"/>
-  <parent link="base_link"/>
-  <child link="rplidar_a1m8_1"/>
-</joint>
 </robot>

Commit message: Arquivo com URDF e transformadas estáticas prontas

File: work_ws/src/salamander_bot/description/robot_core.xacro (robot description, xacro)
@@ -35,12 +35,17 @@
   </collision>
 </link>
+<joint name="chassis_joint" type="fixed">
+  <parent link="base_link"/>
+  <child link="chassis"/>
+  <origin xyz="0.0 0.0 0.0"/>
+</joint>
 <link name="wheel_lf_1">
   <inertial>
-    <origin xyz="6.732011406662686e-09 0.013415334217220576 -2.2496351934075953e-09" rpy="0 0 0"/>
-    <mass value="0.2163222450067834"/>
-    <inertia ixx="8.8e-05" iyy="0.00011" izz="8.8e-05" ixy="0.0" iyz="-0.0" ixz="0.0"/>
+    <origin xyz="0.11315 0.142 -0.03865" rpy="0 0 0"/>
+    <mass value="0.216322"/>
+    <inertia ixx="8.8e-05" iyy="0.00011" izz="8.8e-05" ixy="0.0" iyz="0.0" ixz="0.0"/>
   </inertial>
   <visual>
-    <origin xyz="-0.11315 -0.142 -0.03865" rpy="0 0 0"/>
+    <origin xyz="0 0 0" rpy="0 0 0"/>
     <geometry>
       <mesh filename="file://$(find salamander_bot)/meshes/wheel_lf_1.stl" scale="0.001 0.001 0.001"/>
@@ -49,5 +54,5 @@
   </visual>
   <collision>
-    <origin xyz="-0.11315 -0.142 -0.03865" rpy="0 0 0"/>
+    <origin xyz="0 0 0" rpy="0 0 0"/>
     <geometry>
       <mesh filename="file://$(find salamander_bot)/meshes/wheel_lf_1.stl" scale="0.001 0.001 0.001"/>
@@ -55,12 +60,17 @@
   </collision>
 </link>
+<joint name="wheel_lf_joint" type="continuous">
+  <origin xyz="0.0 0.0 0.0" rpy="0 0 0"/> <parent link="base_link"/>
+  <child link="wheel_lf_1"/>
+  <axis xyz="0.0 1.0 0.0"/>
+</joint>
 <link name="wheel_lb_1">
   <inertial>
-    <origin xyz="3.7014641768307044e-09 0.01344735270580652 -3.504848446189701e-09" rpy="0 0 0"/>
-    <mass value="0.21632224500656735"/>
-    <inertia ixx="8.8e-05" iyy="0.00011" izz="8.8e-05" ixy="-0.0" iyz="-0.0" ixz="0.0"/>
+    <origin xyz="-0.11315 0.142 -0.03865" rpy="0 0 0"/>
+    <mass value="0.216322"/>
+    <inertia ixx="8.8e-05" iyy="0.00011" izz="8.8e-05" ixy="0.0" iyz="0.0" ixz="0.0"/>
   </inertial>
   <visual>
-    <origin xyz="0.11315 -0.142 -0.03865" rpy="0 0 0"/>
+    <origin xyz="0 0 0" rpy="0 0 0"/>
     <geometry>
       <mesh filename="file://$(find salamander_bot)/meshes/wheel_lb_1.stl" scale="0.001 0.001 0.001"/>
@@ -69,5 +79,5 @@
   </visual>
   <collision>
-    <origin xyz="0.11315 -0.142 -0.03865" rpy="0 0 0"/>
+    <origin xyz="0 0 0" rpy="0 0 0"/>
     <geometry>
       <mesh filename="file://$(find salamander_bot)/meshes/wheel_lb_1.stl" scale="0.001 0.001 0.001"/>
@@ -75,12 +85,18 @@
   </collision>
 </link>
+<joint name="wheel_lb_joint" type="continuous">
+  <origin xyz="0.0 0.0 0.0" rpy="0 0 0"/>
+  <parent link="base_link"/>
+  <child link="wheel_lb_1"/>
+  <axis xyz="0.0 1.0 0.0"/>
+</joint>
 <link name="wheel_rf_1">
   <inertial>
-    <origin xyz="6.7541714166008404e-09 -0.013367918230393266 -2.072007607156756e-09" rpy="0 0 0"/>
-    <mass value="0.21632224116980406"/>
-    <inertia ixx="8.8e-05" iyy="0.00011" izz="8.8e-05" ixy="-0.0" iyz="0.0" ixz="0.0"/>
+    <origin xyz="0.11315 -0.142 -0.03865" rpy="0 0 0"/>
+    <mass value="0.216322"/>
+    <inertia ixx="8.8e-05" iyy="0.00011" izz="8.8e-05" ixy="0.0" iyz="0.0" ixz="0.0"/>
   </inertial>
   <visual>
-    <origin xyz="-0.11315 0.142 -0.03865" rpy="0 0 0"/>
+    <origin xyz="0 0 0" rpy="0 0 0"/>
     <geometry>
       <mesh filename="file://$(find salamander_bot)/meshes/wheel_rf_1.stl" scale="0.001 0.001 0.001"/>
@@ -89,5 +105,5 @@
   </visual>
   <collision>
-    <origin xyz="-0.11315 0.142 -0.03865" rpy="0 0 0"/>
+    <origin xyz="0 0 0" rpy="0 0 0"/>
     <geometry>
       <mesh filename="file://$(find salamander_bot)/meshes/wheel_rf_1.stl" scale="0.001 0.001 0.001"/>
@@ -95,12 +111,18 @@
   </collision>
 </link>
+<joint name="wheel_rf_joint" type="continuous">
+  <origin xyz="0.0 0.0 0.0" rpy="0 0 0"/>
+  <parent link="base_link"/>
+  <child link="wheel_rf_1"/>
+  <axis xyz="0.0 1.0 0.0"/>
+</joint>
 <link name="wheel_rb_1">
   <inertial>
-    <origin xyz="3.723448854797695e-09 -0.013447353552784869 -3.327369837990979e-09" rpy="0 0 0"/>
-    <mass value="0.21632224116958718"/>
+    <origin xyz="-0.11315 -0.142 -0.03865" rpy="0 0 0"/>
+    <mass value="0.216322"/>
     <inertia ixx="8.8e-05" iyy="0.00011" izz="8.8e-05" ixy="0.0" iyz="0.0" ixz="0.0"/>
   </inertial>
   <visual>
-    <origin xyz="0.11315 0.142 -0.03865" rpy="0 0 0"/>
+    <origin xyz="0 0 0" rpy="0 0 0"/>
     <geometry>
       <mesh filename="file://$(find salamander_bot)/meshes/wheel_rb_1.stl" scale="0.001 0.001 0.001"/>
@@ -109,5 +131,5 @@
   </visual>
   <collision>
-    <origin xyz="0.11315 0.142 -0.03865" rpy="0 0 0"/>
+    <origin xyz="0 0 0" rpy="0 0 0"/>
     <geometry>
       <mesh filename="file://$(find salamander_bot)/meshes/wheel_rb_1.stl" scale="0.001 0.001 0.001"/>
@@ -115,29 +137,6 @@
   </collision>
 </link>
-<joint name="chassis_joint" type="fixed">
-  <parent link="base_link"/>
-  <child link="chassis"/>
-  <origin xyz="0.0 0.0 0.0"/>
-</joint>
-<joint name="wheel_lf_joint" type="continuous">
-  <origin xyz="0.11315 0.142 0.03865" rpy="0 0 0"/>
-  <parent link="base_link"/>
-  <child link="wheel_lf_1"/>
-  <axis xyz="0.0 1.0 0.0"/>
-</joint>
-<joint name="wheel_lb_joint" type="continuous">
-  <origin xyz="-0.11315 0.142 0.03865" rpy="0 0 0"/>
-  <parent link="base_link"/>
-  <child link="wheel_lb_1"/>
-  <axis xyz="0.0 1.0 0.0"/>
-</joint>
-<joint name="wheel_rf_joint" type="continuous">
-  <origin xyz="0.11315 -0.142 0.03865" rpy="0 0 0"/>
-  <parent link="base_link"/>
-  <child link="wheel_rf_1"/>
-  <axis xyz="0.0 1.0 0.0"/>
-</joint>
 <joint name="wheel_rb_joint" type="continuous">
-  <origin xyz="-0.11315 -0.142 0.03865" rpy="0 0 0"/>
+  <origin xyz="0.0 0.0 0.0" rpy="0 0 0"/>
   <parent link="base_link"/>
   <child link="wheel_rb_1"/>
