Commit message: edicoes-correcao launch

File: work_ws/src/salamander_bot/description/salamander_bot.xacro (robot description, xacro)
@@ -5,4 +5,6 @@
 <xacro:include filename="$(find salamander_bot)/description/salamander_bot.ros2control" />
 <xacro:include filename="$(find salamander_bot)/description/salamander_bot.gazebo" />
+<link name="base_footprint">
+</link>
 <link name="base_link">
   <inertial>
@@ -30,6 +32,4 @@
   <origin xyz="0.0 0.0 0.0" rpy="0.0 0.0 0.0"/>
 </joint>
-<link name="base_footprint">
-</link>
 <!-- Rodas -->
 <link name="wheel_lf_1">
