Commit message: SLAM e edicoes pra simular o lidar

File: work_ws/src/salamander_bot/description/lidar.xacro (robot description, xacro)
@@ -1,24 +1,5 @@
 <?xml version="1.0"?>
 <robot name="salamander_bot" xmlns:xacro="http://www.ros.org/wiki/xacro">
-  <link name="rplidar_a1m8_1">
-    <inertial>
-      <origin xyz="0.0008205477062011579 0.0006535114455110541 0.017493457828168968" rpy="0 0 0"/>
-      <mass value="0.036021408390687064"/>
-      <inertia ixx="1.5e-05" iyy="1.2e-05" izz="2.3e-05" ixy="0.0" iyz="-0.0" ixz="-0.0"/>
-    </inertial>
-    <visual>
-      <origin xyz="0.077204 0.064205 -0.2095" rpy="0 0 0"/>
-      <geometry>
-        <mesh filename="file://$(find salamander_bot)/meshes/rplidar_a1m8_1.stl" scale="0.001 0.001 0.001"/>
-      </geometry>
-      <material name="blue"/>
-    </visual>
-    <collision>
-      <origin xyz="0.077204 0.064205 -0.2095" rpy="0 0 0"/>
-      <geometry>
-        <mesh filename="file://$(find salamander_bot)/meshes/rplidar_a1m8_1.stl" scale="0.001 0.001 0.001"/>
-      </geometry>
-    </collision>
-  </link>
+<!-- Lidar joint -->
 <joint name="rplidar_a1m8_joint" type="fixed">
   <origin xyz="-0.077204 -0.064205 0.2095" rpy="0 0 0"/>
@@ -26,10 +7,31 @@
   <child link="rplidar_a1m8_1"/>
 </joint>
+<!-- Lidar frame -->
+<link name="rplidar_a1m8_1">
+  <inertial>
+    <origin xyz="0.0008205477062011579 0.0006535114455110541 0.017493457828168968" rpy="0 0 0"/>
+    <mass value="0.036021408390687064"/>
+    <inertia ixx="1.5e-05" iyy="1.2e-05" izz="2.3e-05" ixy="0.0" iyz="-0.0" ixz="-0.0"/>
+  </inertial>
+  <visual>
+    <origin xyz="0.077204 0.064205 -0.2095" rpy="0 0 0"/>
+    <geometry>
+      <mesh filename="file://$(find salamander_bot)/meshes/rplidar_a1m8_1.stl" scale="0.001 0.001 0.001"/>
+    </geometry>
+    <material name="blue"/>
+  </visual>
+  <collision>
+    <origin xyz="0.077204 0.064205 -0.2095" rpy="0 0 0"/>
+    <geometry>
+      <mesh filename="file://$(find salamander_bot)/meshes/rplidar_a1m8_1.stl" scale="0.001 0.001 0.001"/>
+    </geometry>
+  </collision>
+</link>
 <gazebo reference="rplidar_a1m8_1">
-  <sensor name="lidar_sensor" type="gpu_lidar">
+  <sensor name="lidar" type="gpu_lidar">
     <pose>0 0 0 0 0 0</pose>
     <update_rate>10</update_rate>
     <visualize>true</visualize>
-    <topic>scan</topic>
+    <topic>/scan</topic>
     <lidar>
       <scan>
@@ -42,9 +44,9 @@
       </scan>
       <range>
-        <min>0.3</min>
+        <min>0.15</min>
         <max>12.0</max>
-        <resolution>0.01</resolution>
       </range>
     </lidar>
+    <gz_frame_id>rplidar_a1m8_1</gz_frame_id>
     <always_on>true</always_on>
   </sensor>

File: work_ws/src/salamander_bot/description/robot_core.xacro (robot description, xacro)
@@ -4,5 +4,15 @@
 <xacro:include filename="$(find salamander_bot)/description/salamander_bot.ros2control" />
 <xacro:include filename="$(find salamander_bot)/description/salamander_bot.gazebo" />
-<link name="base_link"></link>
+<!-- Adicionado SLAM -->
+<link name="base_link">
+</link>
+<joint name="base_footprint_joint" type="fixed">
+  <parent link="base_link"/>
+  <child link="base_footprint"/>
+  <origin xyz="0.0 0.0 0.0" rpy="0.0 0.0 0.0"/>
+</joint>
+<link name="base_footprint">
+</link>
+<!-- fim SLAM -->
 <link name="chassis">
   <inertial>

Commit message: Merge URDF-Nav-Map

File: work_ws/src/salamander_bot/description/lidar.xacro (robot description, xacro)
@@ -2,6 +2,6 @@
 <robot name="salamander_bot" xmlns:xacro="http://www.ros.org/wiki/xacro">
 <!-- Lidar joint -->
-<joint name="rplidar_a1m8_joint" type="fixed">
-  <origin xyz="-0.077204 -0.064205 0.2095" rpy="0 0 0"/>
+<joint name="Rigid 11" type="fixed">
+  <origin xyz="0.236098 -0.004646 0.000956" rpy="0 0 0"/>
   <parent link="base_link"/>
   <child link="rplidar_a1m8_1"/>
@@ -10,17 +10,17 @@
 <link name="rplidar_a1m8_1">
   <inertial>
-    <origin xyz="0.0008205477062011579 0.0006535114455110541 0.017493457828168968" rpy="0 0 0"/>
+    <origin xyz="-0.016984302698711456 0.004773780112382523 0.02905054217183256" rpy="0 0 0"/>
     <mass value="0.036021408390687064"/>
-    <inertia ixx="1.5e-05" iyy="1.2e-05" izz="2.3e-05" ixy="0.0" iyz="-0.0" ixz="-0.0"/>
+    <inertia ixx="1.5e-05" iyy="1.2e-05" izz="2.3e-05" ixy="-0.0" iyz="0.0" ixz="-0.0"/>
   </inertial>
   <visual>
-    <origin xyz="0.077204 0.064205 -0.2095" rpy="0 0 0"/>
+    <origin xyz="-0.236098 0.004646 -0.000956" rpy="0 0 0"/>
     <geometry>
       <mesh filename="file://$(find salamander_bot)/meshes/rplidar_a1m8_1.stl" scale="0.001 0.001 0.001"/>
     </geometry>
-    <material name="blue"/>
+    <material name="silver"/>
   </visual>
   <collision>
-    <origin xyz="0.077204 0.064205 -0.2095" rpy="0 0 0"/>
+    <origin xyz="-0.236098 0.004646 -0.000956" rpy="0 0 0"/>
     <geometry>
       <mesh filename="file://$(find salamander_bot)/meshes/rplidar_a1m8_1.stl" scale="0.001 0.001 0.001"/>

File: work_ws/src/salamander_bot/description/salamander_bot.xacro (robot description, xacro)
@@ -1,7 +1,7 @@
 <?xml version="1.0" ?>
 <robot name="salamander_bot" xmlns:xacro="http://www.ros.org/wiki/xacro">
-<xacro:include filename="$(find salamander_bot_description)/urdf/materials.xacro" />
-<xacro:include filename="$(find salamander_bot_description)/urdf/salamander_bot.ros2control" />
-<xacro:include filename="$(find salamander_bot_description)/urdf/salamander_bot.gazebo" />
+<xacro:include filename="$(find salamander_bot)/description/materials.xacro" />
+<xacro:include filename="$(find salamander_bot)/description/salamander_bot.ros2control" />
+<xacro:include filename="$(find salamander_bot)/description/salamander_bot.gazebo" />
 <link name="base_link">
   <inertial>
@@ -13,5 +13,5 @@
     <origin xyz="0 0 0" rpy="0 0 0"/>
     <geometry>
-      <mesh filename="file://$(find salamander_bot_description)/meshes/base_link.stl" scale="0.001 0.001 0.001"/>
+      <mesh filename="file://$(find salamander_bot)/description/meshes/base_link.stl" scale="0.001 0.001 0.001"/>
     </geometry>
     <material name="silver"/>
@@ -20,7 +20,14 @@
     <origin xyz="0 0 0" rpy="0 0 0"/>
     <geometry>
-      <mesh filename="file://$(find salamander_bot_description)/meshes/base_link.stl" scale="0.001 0.001 0.001"/>
+      <mesh filename="file://$(find salamander_bot)/meshes/base_link.stl" scale="0.001 0.001 0.001"/>
     </geometry>
   </collision>
+</link>
+<joint name="base_footprint_joint" type="fixed">
+  <parent link="base_link"/>
+  <child link="base_footprint"/>
+  <origin xyz="0.0 0.0 0.0" rpy="0.0 0.0 0.0"/>
+</joint>
+<link name="base_footprint">
 </link>
 <link name="wheel_lf_1">
@@ -33,5 +40,5 @@
     <origin xyz="-0.11315 -0.142 -0.03865" rpy="0 0 0"/>
     <geometry>
-      <mesh filename="file://$(find salamander_bot_description)/meshes/wheel_lf_1.stl" scale="0.001 0.001 0.001"/>
+      <mesh filename="file://$(find salamander_bot)/meshes/wheel_lf_1.stl" scale="0.001 0.001 0.001"/>
     </geometry>
     <material name="silver"/>
@@ -40,5 +47,5 @@
     <origin xyz="-0.11315 -0.142 -0.03865" rpy="0 0 0"/>
     <geometry>
-      <mesh filename="file://$(find salamander_bot_description)/meshes/wheel_lf_1.stl" scale="0.001 0.001 0.001"/>
+      <mesh filename="file://$(find salamander_bot)/meshes/wheel_lf_1.stl" scale="0.001 0.001 0.001"/>
     </geometry>
   </collision>
@@ -53,5 +60,5 @@
     <origin xyz="0.11315 -0.142 -0.03865" rpy="0 0 0"/>
     <geometry>
-      <mesh filename="file://$(find salamander_bot_description)/meshes/wheel_lb_1.stl" scale="0.001 0.001 0.001"/>
+      <mesh filename="file://$(find salamander_bot)/meshes/wheel_lb_1.stl" scale="0.001 0.001 0.001"/>
     </geometry>
     <material name="silver"/>
@@ -60,5 +67,5 @@
     <origin xyz="0.11315 -0.142 -0.03865" rpy="0 0 0"/>
     <geometry>
-      <mesh filename="file://$(find salamander_bot_description)/meshes/wheel_lb_1.stl" scale="0.001 0.001 0.001"/>
+      <mesh filename="file://$(find salamander_bot)/meshes/wheel_lb_1.stl" scale="0.001 0.001 0.001"/>
     </geometry>
   </collision>
@@ -73,5 +80,5 @@
     <origin xyz="-0.11315 0.142 -0.03865" rpy="0 0 0"/>
     <geometry>
-      <mesh filename="file://$(find salamander_bot_description)/meshes/wheel_rf_1.stl" scale="0.001 0.001 0.001"/>
+      <mesh filename="file://$(find salamander_bot)/meshes/wheel_rf_1.stl" scale="0.001 0.001 0.001"/>
     </geometry>
     <material name="silver"/>
@@ -80,5 +87,5 @@
     <origin xyz="-0.11315 0.142 -0.03865" rpy="0 0 0"/>
     <geometry>
-      <mesh filename="file://$(find salamander_bot_description)/meshes/wheel_rf_1.stl" scale="0.001 0.001 0.001"/>
+      <mesh filename="file://$(find salamander_bot)/meshes/wheel_rf_1.stl" scale="0.001 0.001 0.001"/>
     </geometry>
   </collision>
@@ -93,5 +100,5 @@
     <origin xyz="0.11315 0.142 -0.03865" rpy="0 0 0"/>
     <geometry>
-      <mesh filename="file://$(find salamander_bot_description)/meshes/wheel_rb_1.stl" scale="0.001 0.001 0.001"/>
+      <mesh filename="file://$(find salamander_bot)/meshes/wheel_rb_1.stl" scale="0.001 0.001 0.001"/>
     </geometry>
     <material name="silver"/>
@@ -100,25 +107,5 @@
     <origin xyz="0.11315 0.142 -0.03865" rpy="0 0 0"/>
     <geometry>
-      <mesh filename="file://$(find salamander_bot_description)/meshes/wheel_rb_1.stl" scale="0.001 0.001 0.001"/>
-    </geometry>
-  </collision>
-</link>
-<link name="rplidar_a1m8_1">
-  <inertial>
-    <origin xyz="-0.016984302698711456 0.004773780112382523 0.02905054217183256" rpy="0 0 0"/>
-    <mass value="0.036021408390687064"/>
-    <inertia ixx="1.5e-05" iyy="1.2e-05" izz="2.3e-05" ixy="-0.0" iyz="0.0" ixz="-0.0"/>
-  </inertial>
-  <visual>
-    <origin xyz="-0.236098 0.004646 -0.000956" rpy="0 0 0"/>
-    <geometry>
-      <mesh filename="file://$(find salamander_bot_description)/meshes/rplidar_a1m8_1.stl" scale="0.001 0.001 0.001"/>
-    </geometry>
-    <material name="silver"/>
-  </visual>
-  <collision>
-    <origin xyz="-0.236098 0.004646 -0.000956" rpy="0 0 0"/>
-    <geometry>
-      <mesh filename="file://$(find salamander_bot_description)/meshes/rplidar_a1m8_1.stl" scale="0.001 0.001 0.001"/>
+      <mesh filename="file://$(find salamander_bot)/meshes/wheel_rb_1.stl" scale="0.001 0.001 0.001"/>
     </geometry>
   </collision>
@@ -148,8 +135,3 @@
   <axis xyz="-0.0 -1.0 0.0"/>
 </joint>
-<joint name="Rigid 11" type="fixed">
-  <origin xyz="0.236098 -0.004646 0.000956" rpy="0 0 0"/>
-  <parent link="base_link"/>
-  <child link="rplidar_a1m8_1"/>
-</joint>
 </robot>

Commit message: limpeza build install e log + edição xacros

File: work_ws/src/salamander_bot/description/lidar.xacro (robot description, xacro)
@@ -2,5 +2,5 @@
 <robot name="salamander_bot" xmlns:xacro="http://www.ros.org/wiki/xacro">
 <!-- Lidar joint -->
-<joint name="Rigid 11" type="fixed">
+<joint name="rplidar_a1m8_joint" type="fixed">
   <origin xyz="0.236098 -0.004646 0.000956" rpy="0 0 0"/>
   <parent link="base_link"/>

File: work_ws/src/salamander_bot/description/salamander_bot.xacro (robot description, xacro)
@@ -1,5 +1,5 @@
 <?xml version="1.0" ?>
 <robot name="salamander_bot" xmlns:xacro="http://www.ros.org/wiki/xacro">
-<xacro:include filename="$(find salamander_bot)/description/materials.xacro" />
+<xacro:include filename="$(find salamander_bot)/description/colors.xacro" />
 <xacro:include filename="$(find salamander_bot)/description/salamander_bot.ros2control" />
 <xacro:include filename="$(find salamander_bot)/description/salamander_bot.gazebo" />
@@ -13,5 +13,5 @@
     <origin xyz="0 0 0" rpy="0 0 0"/>
     <geometry>
-      <mesh filename="file://$(find salamander_bot)/description/meshes/base_link.stl" scale="0.001 0.001 0.001"/>
+      <mesh filename="file://$(find salamander_bot)/meshes/base_link.stl" scale="0.001 0.001 0.001"/>
     </geometry>
     <material name="silver"/>

Commit message: simulação do lidar no gazebo

File: work_ws/src/salamander_bot/description/lidar.xacro (robot description, xacro)
@@ -28,27 +28,3 @@
   </collision>
 </link>
-<gazebo reference="rplidar_a1m8_1">
-  <sensor name="lidar" type="lidar">
-    <pose>0 0 0 0 0 0</pose>
-    <update_rate>10</update_rate>
-    <visualize>false</visualize>
-    <topic>/sim/scan</topic>
-    <lidar>
-      <scan>
-        <horizontal>
-          <samples>360</samples>
-          <resolution>1</resolution>
-          <min_angle>-3.14</min_angle>
-          <max_angle>3.14</max_angle>
-        </horizontal>
-      </scan>
-      <range>
-        <min>0.15</min>
-        <max>12.0</max>
-      </range>
-    </lidar>
-    <gz_frame_id>rplidar_a1m8_1</gz_frame_id>
-    <always_on>true</always_on>
-  </sensor>
-</gazebo>
 </robot>

File: work_ws/src/salamander_bot/description/robot.urdf.xacro (robot description, xacro)
@@ -2,6 +2,4 @@
 <robot name="salamander_bot" xmlns:xacro="http://www.ros.org/wiki/xacro">
     <!-- Robot Core File -->
-    <xacro:include filename="robot_core.xacro" />
-    <!-- Lidar -->
-    <xacro:include filename="lidar.xacro" />
+    <xacro:include filename="salamander_bot.xacro" />
 </robot>

File: work_ws/src/salamander_bot/description/salamander_bot.xacro (robot description, xacro)
@@ -2,4 +2,5 @@
 <robot name="salamander_bot" xmlns:xacro="http://www.ros.org/wiki/xacro">
 <xacro:include filename="$(find salamander_bot)/description/colors.xacro" />
+<xacro:include filename="$(find salamander_bot)/description/lidar.xacro" />
 <xacro:include filename="$(find salamander_bot)/description/salamander_bot.ros2control" />
 <xacro:include filename="$(find salamander_bot)/description/salamander_bot.gazebo" />
@@ -24,11 +25,12 @@
   </collision>
 </link>
-<joint name="base_footprint_joint" type="fixed">
-  <parent link="base_link"/>
-  <child link="base_footprint"/>
+<joint name="base_link_joint" type="fixed">
+  <parent link="base_footprint"/>
+  <child link="base_link"/>
   <origin xyz="0.0 0.0 0.0" rpy="0.0 0.0 0.0"/>
 </joint>
 <link name="base_footprint">
 </link>
+<!-- Rodas -->
 <link name="wheel_lf_1">
   <inertial>
@@ -111,5 +113,5 @@
   </collision>
 </link>
-<joint name="wheel_lf_joint" type="continuous">
+<joint name="wheel_lf_1_joint" type="continuous">
   <origin xyz="0.11315 0.142 0.03865" rpy="0 0 0"/>
   <parent link="base_link"/>
@@ -117,5 +119,5 @@
   <axis xyz="0.0 1.0 -0.0"/>
 </joint>
-<joint name="wheel_lb_joint" type="continuous">
+<joint name="wheel_lb_1_joint" type="continuous">
   <origin xyz="-0.11315 0.142 0.03865" rpy="0 0 0"/>
   <parent link="base_link"/>
@@ -123,5 +125,5 @@
   <axis xyz="-0.0 1.0 -0.0"/>
 </joint>
-<joint name="wheel_rf_joint" type="continuous">
+<joint name="wheel_rf_1_joint" type="continuous">
   <origin xyz="0.11315 -0.142 0.03865" rpy="0 0 0"/>
   <parent link="base_link"/>
@@ -129,5 +131,5 @@
   <axis xyz="-0.0 -1.0 0.0"/>
 </joint>
-<joint name="wheel_rb_joint" type="continuous">
+<joint name="wheel_rb_1_joint" type="continuous">
   <origin xyz="-0.11315 -0.142 0.03865" rpy="0 0 0"/>
   <parent link="base_link"/>

Commit message: Nav2 funcionando, params lidar.xacro modificados

File: work_ws/src/salamander_bot/description/lidar.xacro (robot description, xacro)
@@ -3,5 +3,5 @@
 <!-- Lidar joint -->
 <joint name="rplidar_a1m8_joint" type="fixed">
-  <origin xyz="0.236098 -0.004646 0.000956" rpy="0 0 0"/>
+  <origin xyz="0.236098 -0.004646 0.000956" rpy="3.14159 0 1.5708"/> #o valor foi ajustado para que o Lidar fique na posição correta em relação ao robô, considerando a orientação e a posição do sensor em relação à base do robô.
   <parent link="base_link"/>
   <child link="rplidar_a1m8_1"/>
