Commit message: Adicionado URDF Inicial de Robô Final (Manipulador + Chassi + Câmera + LIDAR) (Corrigir Câmera e LIDAR) & Correção na Modelagem da Cinemática Inversa da Movimentação - ESTAVA EM RAD/S AO INVÉS DE M/S :(((( (TESTAR)

File: work_ws/src/salamander_bot/description/lidar.xacro (robot description, xacro)
@@ -1,5 +1,16 @@
 <?xml version="1.0"?>
 <robot name="salamander_bot" xmlns:xacro="http://www.ros.org/wiki/xacro">
+<<<<<<< HEAD
 <link name="rplidar_a1m8">
+=======
+<!-- Lidar joint -->
+<joint name="rplidar_a1m8_joint" type="fixed">
+  <origin xyz="0.236098 -0.004646 0.000956" rpy="0 0 0"/>
+  <parent link="base_link"/>
+  <child link="rplidar_a1m8_1"/>
+</joint>
+<!-- Lidar frame -->
+<link name="rplidar_a1m8_1">
+>>>>>>> 473ca78 (Adicionado URDF Inicial de Robô Final (Manipulador + Chassi + Câmera + LIDAR) (Corrigir Câmera e LIDAR) & Correção na Modelagem da Cinemática Inversa da Movimentação - ESTAVA EM RAD/S AO INVÉS DE M/S :(((( (TESTAR))
   <inertial>
     <origin xyz="219.933902e-03 -0.526156e-03 29.599964e-03" rpy="0 0 0"/>
@@ -8,5 +19,9 @@
   </inertial>
   <visual>
+<<<<<<< HEAD
     <origin xyz="0 0 0" rpy="0 0 0"/>
+=======
+    <origin xyz="-0.236098 0.004646 -0.000956" rpy="0.0 0 0"/>
+>>>>>>> 473ca78 (Adicionado URDF Inicial de Robô Final (Manipulador + Chassi + Câmera + LIDAR) (Corrigir Câmera e LIDAR) & Correção na Modelagem da Cinemática Inversa da Movimentação - ESTAVA EM RAD/S AO INVÉS DE M/S :(((( (TESTAR))
     <geometry>
       <cylinder length="0.0235" radius="0.035075" />
@@ -15,5 +30,9 @@
   </visual>
   <collision>
+<<<<<<< HEAD
     <origin xyz="0 0 0" rpy="0 0 0"/>
+=======
+    <origin xyz="-0.236098 0.004646 -0.000956" rpy="0.0 0 0"/>
+>>>>>>> 473ca78 (Adicionado URDF Inicial de Robô Final (Manipulador + Chassi + Câmera + LIDAR) (Corrigir Câmera e LIDAR) & Correção na Modelagem da Cinemática Inversa da Movimentação - ESTAVA EM RAD/S AO INVÉS DE M/S :(((( (TESTAR))
     <geometry>
       <cylinder length="0.0235" radius="0.035075" />

File: work_ws/src/salamander_bot/description/salamander_bot.xacro (robot description, xacro)
@@ -2,5 +2,7 @@
 <robot name="salamander_bot" xmlns:xacro="http://www.ros.org/wiki/xacro">
 <xacro:include filename="$(find salamander_bot)/description/colors.xacro" />
+<xacro:include filename="$(find salamander_bot)/description/arm_platform.xacro" />
 <xacro:include filename="$(find salamander_bot)/description/lidar.xacro" />
+<xacro:include filename="$(find salamander_bot)/description/webcam.xacro" />
 <xacro:include filename="$(find salamander_bot)/description/salamander_bot.ros2control" />
 <xacro:include filename="$(find salamander_bot)/description/salamander_bot.gazebo" />

Commit message: Adicionado URDF Inicial de Robô Final (Manipulador + Chassi + Câmera + LIDAR) (Corrigir Câmera e LIDAR) & Correção na Modelagem da Cinemática Inversa da Movimentação - ESTAVA EM RAD/S AO INVÉS DE M/S :(((( (TESTAR)

File: work_ws/src/salamander_bot/description/lidar.xacro (robot description, xacro)
@@ -3,5 +3,5 @@
 <!-- Lidar joint -->
 <joint name="rplidar_a1m8_joint" type="fixed">
-  <origin xyz="0.236098 -0.004646 0.000956" rpy="3.14159 0 1.5708"/> #o valor foi ajustado para que o Lidar fique na posição correta em relação ao robô, considerando a orientação e a posição do sensor em relação à base do robô.
+  <origin xyz="0.236098 -0.004646 0.000956" rpy="0 0 0"/>
   <parent link="base_link"/>
   <child link="rplidar_a1m8_1"/>
@@ -15,5 +15,5 @@
   </inertial>
   <visual>
-    <origin xyz="-0.236098 0.004646 -0.000956" rpy="0 0 0"/>
+    <origin xyz="-0.236098 0.004646 -0.000956" rpy="0.0 0 0"/>
     <geometry>
       <mesh filename="file://$(find salamander_bot)/meshes/rplidar_a1m8_1.stl" scale="0.001 0.001 0.001"/>
@@ -22,5 +22,5 @@
   </visual>
   <collision>
-    <origin xyz="-0.236098 0.004646 -0.000956" rpy="0 0 0"/>
+    <origin xyz="-0.236098 0.004646 -0.000956" rpy="0.0 0 0"/>
     <geometry>
       <mesh filename="file://$(find salamander_bot)/meshes/rplidar_a1m8_1.stl" scale="0.001 0.001 0.001"/>

File: work_ws/src/salamander_bot/description/salamander_bot.xacro (robot description, xacro)
@@ -2,5 +2,7 @@
 <robot name="salamander_bot" xmlns:xacro="http://www.ros.org/wiki/xacro">
 <xacro:include filename="$(find salamander_bot)/description/colors.xacro" />
+<xacro:include filename="$(find salamander_bot)/description/arm_platform.xacro" />
 <xacro:include filename="$(find salamander_bot)/description/lidar.xacro" />
+<xacro:include filename="$(find salamander_bot)/description/webcam.xacro" />
 <xacro:include filename="$(find salamander_bot)/description/salamander_bot.ros2control" />
 <xacro:include filename="$(find salamander_bot)/description/salamander_bot.gazebo" />

Commit message: Reorganização de Arquivos URDF do Chassi, Posições de Frames Atualizados, Simplificação no Modelo de Colisão (Ainda tem Muita Coisa a Ajustar com Relação ao Visual), Alteração da Posição X,Y das Rodas na Convenção Correta.

File: work_ws/src/salamander_bot/description/lidar.xacro (robot description, xacro)
@@ -1,12 +1,5 @@
 <?xml version="1.0"?>
 <robot name="salamander_bot" xmlns:xacro="http://www.ros.org/wiki/xacro">
-<!-- Lidar joint -->
-<joint name="rplidar_a1m8_joint" type="fixed">
-  <origin xyz="0.236098 -0.004646 0.000956" rpy="0 0 0"/>
-  <parent link="base_link"/>
-  <child link="rplidar_a1m8_1"/>
-</joint>
-<!-- Lidar frame -->
-<link name="rplidar_a1m8_1">
+<link name="rplidar_a1m8">
   <inertial>
     <origin xyz="-0.016984302698711456 0.004773780112382523 0.02905054217183256" rpy="0 0 0"/>
@@ -15,16 +8,21 @@
   </inertial>
   <visual>
-    <origin xyz="-0.236098 0.004646 -0.000956" rpy="0.0 0 0"/>
+    <origin xyz="-219.933902e-03 0.526156e-03 -29.599964e-03" rpy="0 0 0"/>
     <geometry>
-      <mesh filename="file://$(find salamander_bot)/meshes/rplidar_a1m8_1.stl" scale="0.001 0.001 0.001"/>
+      <mesh filename="file://$(find salamander_bot)/meshes/rplidar_a1m8.stl" scale="0.001 0.001 0.001"/>
     </geometry>
     <material name="silver"/>
   </visual>
   <collision>
-    <origin xyz="-0.236098 0.004646 -0.000956" rpy="0.0 0 0"/>
+    <origin xyz="0 0 0" rpy="0 0 0"/>
     <geometry>
-      <mesh filename="file://$(find salamander_bot)/meshes/rplidar_a1m8_1.stl" scale="0.001 0.001 0.001"/>
+      <cylinder length="0.0235" radius="0.035075" />
     </geometry>
   </collision>
 </link>
+<joint name="rplidar_a1m8_joint" type="fixed">
+  <parent link="base_link"/>
+  <child link="rplidar_a1m8"/>
+  <origin xyz="219.933902e-03 -0.526156e-03 -10.400036e-03" rpy="0 0 0"/>
+</joint>
 </robot>

File: work_ws/src/salamander_bot/description/salamander_bot.xacro (robot description, xacro)
@@ -16,5 +16,5 @@
   </inertial>
   <visual>
-    <origin xyz="0 0 0" rpy="0 0 0"/>
+    <origin xyz="16.16414e-03 -4.12017e-03 -79.543971e-03" rpy="0 0 0"/>
     <geometry>
       <mesh filename="package://salamander_bot/meshes/base_link.stl" scale="0.001 0.001 0.001"/>
@@ -23,7 +23,87 @@
   </visual>
   <collision>
-    <origin xyz="0 0 0" rpy="0 0 0"/>
+    <origin xyz="16.16414e-03 -4.12017e-03 -79.543971e-03" rpy="0 0 0"/>
     <geometry>
-      <mesh filename="package://salamander_bot/meshes/base_link.stl" scale="0.001 0.001 0.001"/>
+      <mesh filename="package://salamander_bot/meshes/base_link_collision.stl" scale="0.001 0.001 0.001"/>
+    </geometry>
+  </collision>
+</link>
+<link name="wheel_lf">
+  <inertial>
+    <origin xyz="6.732011406662686e-09 0.013415334217220576 -2.2496351934075953e-09" rpy="0 0 0"/>
+    <mass value="0.2163222450067834"/>
+    <inertia ixx="8.8e-05" iyy="0.00011" izz="8.8e-05" ixy="0.0" iyz="-0.0" ixz="0.0"/>
+  </inertial>
+  <visual>
+    <origin xyz="-113.15e-03 -148.75e-03 -40.00e-03" rpy="0 0 0"/>
+    <geometry>
+      <mesh filename="package://salamander_bot/meshes/wheel_lf.stl" scale="0.001 0.001 0.001"/>
+    </geometry>
+    <material name="silver"/>
+  </visual>
+  <collision>
+    <origin xyz="0 0 0" rpy="${pi/2} 0 0"/>
+    <geometry>
+      <cylinder length="0.0375" radius="0.04" />
+    </geometry>
+  </collision>
+</link>
+<link name="wheel_lb">
+  <inertial>
+    <origin xyz="3.7014641768307044e-09 0.01344735270580652 -3.504848446189701e-09" rpy="0 0 0"/>
+    <mass value="0.21632224500656735"/>
+    <inertia ixx="8.8e-05" iyy="0.00011" izz="8.8e-05" ixy="-0.0" iyz="-0.0" ixz="0.0"/>
+  </inertial>
+  <visual>
+    <origin xyz="113.15e-03 -148.75e-03 -40.00e-03" rpy="0 0 0"/>
+    <geometry>
+      <mesh filename="package://salamander_bot/meshes/wheel_lb.stl" scale="0.001 0.001 0.001"/>
+    </geometry>
+    <material name="silver"/>
+  </visual>
+  <collision>
+    <origin xyz="0 0 0" rpy="${pi/2} 0 0"/>
+    <geometry>
+      <cylinder length="0.0375" radius="0.04" />
+    </geometry>
+  </collision>
+</link>
+<link name="wheel_rf">
+  <inertial>
+    <origin xyz="6.7541714166008404e-09 -0.013367918230393266 -2.072007607156756e-09" rpy="0 0 0"/>
+    <mass value="0.21632224116980406"/>
+    <inertia ixx="8.8e-05" iyy="0.00011" izz="8.8e-05" ixy="-0.0" iyz="0.0" ixz="0.0"/>
+  </inertial>
+  <visual>
+    <origin xyz="-113.15e-03 148.75e-03 -40.00e-03" rpy="0 0 0"/>
+    <geometry>
+      <mesh filename="package://salamander_bot/meshes/wheel_rf.stl" scale="0.001 0.001 0.001"/>
+    </geometry>
+    <material name="silver"/>
+  </visual>
+  <collision>
+    <origin xyz="0 0 0" rpy="${pi/2} 0 0"/>
+    <geometry>
+      <cylinder length="0.0375" radius="0.04" />
+    </geometry>
+  </collision>
+</link>
+<link name="wheel_rb">
+  <inertial>
+    <origin xyz="3.723448854797695e-09 -0.013447353552784869 -3.327369837990979e-09" rpy="0 0 0"/>
+    <mass value="0.21632224116958718"/>
+    <inertia ixx="8.8e-05" iyy="0.00011" izz="8.8e-05" ixy="0.0" iyz="0.0" ixz="0.0"/>
+  </inertial>
+  <visual>
+    <origin xyz="113.15e-03 148.75e-03 -40.00e-03" rpy="0 0 0"/>
+    <geometry>
+      <mesh filename="package://salamander_bot/meshes/wheel_rb.stl" scale="0.001 0.001 0.001"/>
+    </geometry>
+    <material name="silver"/>
+  </visual>
+  <collision>
+    <origin xyz="0 0 0" rpy="${pi/2} 0 0"/>
+    <geometry>
+      <cylinder length="0.0375" radius="0.04" />
     </geometry>
   </collision>
@@ -32,110 +112,29 @@
   <parent link="base_footprint"/>
   <child link="base_link"/>
-  <origin xyz="0.0 0.0 0.0" rpy="0.0 0.0 0.0"/>
+  <origin xyz="0.0 0.0 40.0e-03" rpy="0.0 0.0 0.0"/>
 </joint>
-<!-- Rodas -->
-<link name="wheel_lf_1">
-  <inertial>
-    <origin xyz="6.732011406662686e-09 0.013415334217220576 -2.2496351934075953e-09" rpy="0 0 0"/>
-    <mass value="0.2163222450067834"/>
-    <inertia ixx="8.8e-05" iyy="0.00011" izz="8.8e-05" ixy="0.0" iyz="-0.0" ixz="0.0"/>
-  </inertial>
-  <visual>
-    <origin xyz="-0.11315 -0.142 -0.03865" rpy="0 0 0"/>
-    <geometry>
-      <mesh filename="package://salamander_bot/meshes/wheel_lf_1.stl" scale="0.001 0.001 0.001"/>
-    </geometry>
-    <material name="silver"/>
-  </visual>
-  <collision>
-    <origin xyz="-0.11315 -0.142 -0.03865" rpy="0 0 0"/>
-    <geometry>
-      <mesh filename="package://salamander_bot/meshes/wheel_lf_1.stl" scale="0.001 0.001 0.001"/>
-    </geometry>
-  </collision>
-</link>
-<link name="wheel_lb_1">
-  <inertial>
-    <origin xyz="3.7014641768307044e-09 0.01344735270580652 -3.504848446189701e-09" rpy="0 0 0"/>
-    <mass value="0.21632224500656735"/>
-    <inertia ixx="8.8e-05" iyy="0.00011" izz="8.8e-05" ixy="-0.0" iyz="-0.0" ixz="0.0"/>
-  </inertial>
-  <visual>
-    <origin xyz="0.11315 -0.142 -0.03865" rpy="0 0 0"/>
-    <geometry>
-      <mesh filename="package://salamander_bot/meshes/wheel_lb_1.stl" scale="0.001 0.001 0.001"/>
-    </geometry>
-    <material name="silver"/>
-  </visual>
-  <collision>
-    <origin xyz="0.11315 -0.142 -0.03865" rpy="0 0 0"/>
-    <geometry>
-      <mesh filename="package://salamander_bot/meshes/wheel_lb_1.stl" scale="0.001 0.001 0.001"/>
-    </geometry>
-  </collision>
-</link>
-<link name="wheel_rf_1">
-  <inertial>
-    <origin xyz="6.7541714166008404e-09 -0.013367918230393266 -2.072007607156756e-09" rpy="0 0 0"/>
-    <mass value="0.21632224116980406"/>
-    <inertia ixx="8.8e-05" iyy="0.00011" izz="8.8e-05" ixy="-0.0" iyz="0.0" ixz="0.0"/>
-  </inertial>
-  <visual>
-    <origin xyz="-0.11315 0.142 -0.03865" rpy="0 0 0"/>
-    <geometry>
-      <mesh filename="package://salamander_bot/meshes/wheel_rf_1.stl" scale="0.001 0.001 0.001"/>
-    </geometry>
-    <material name="silver"/>
-  </visual>
-  <collision>
-    <origin xyz="-0.11315 0.142 -0.03865" rpy="0 0 0"/>
-    <geometry>
-      <mesh filename="package://salamander_bot/meshes/wheel_rf_1.stl" scale="0.001 0.001 0.001"/>
-    </geometry>
-  </collision>
-</link>
-<link name="wheel_rb_1">
-  <inertial>
-    <origin xyz="3.723448854797695e-09 -0.013447353552784869 -3.327369837990979e-09" rpy="0 0 0"/>
-    <mass value="0.21632224116958718"/>
-    <inertia ixx="8.8e-05" iyy="0.00011" izz="8.8e-05" ixy="0.0" iyz="0.0" ixz="0.0"/>
-  </inertial>
-  <visual>
-    <origin xyz="0.11315 0.142 -0.03865" rpy="0 0 0"/>
-    <geometry>
-      <mesh filename="package://salamander_bot/meshes/wheel_rb_1.stl" scale="0.001 0.001 0.001"/>
-    </geometry>
-    <material name="silver"/>
-  </visual>
-  <collision>
-    <origin xyz="0.11315 0.142 -0.03865" rpy="0 0 0"/>
-    <geometry>
-      <mesh filename="package://salamander_bot/meshes/wheel_rb_1.stl" scale="0.001 0.001 0.001"/>
-    </geometry>
-  </collision>
-</link>
-<joint name="wheel_lf_1_joint" type="continuous">
-  <origin xyz="0.11315 0.142 0.03865" rpy="0 0 0"/>
+<joint name="wheel_lf_joint" type="continuous">
+  <origin xyz="113.15e-03 148.75e-03 0.0" rpy="0 0 0"/>
   <parent link="base_link"/>
-  <child link="wheel_lf_1"/>
-  <axis xyz="0.0 1.0 -0.0"/>
+  <child link="wheel_lf"/>
+  <axis xyz="0.0 1.0 0.0"/>
 </joint>
-<joint name="wheel_lb_1_joint" type="continuous">
-  <origin xyz="-0.11315 0.142 0.03865" rpy="0 0 0"/>
+<joint name="wheel_lb_joint" type="continuous">
+  <origin xyz="-113.15e-03 148.75e-03 0.0" rpy="0 0 0"/>
   <parent link="base_link"/>
-  <child link="wheel_lb_1"/>
-  <axis xyz="-0.0 1.0 -0.0"/>
+  <child link="wheel_lb"/>
+  <axis xyz="0.0 1.0 0.0"/>
 </joint>
-<joint name="wheel_rf_1_joint" type="continuous">
-  <origin xyz="0.11315 -0.142 0.03865" rpy="0 0 0"/>
+<joint name="wheel_rf_joint" type="continuous">
+  <origin xyz="113.15e-03 -148.75e-03 0.0" rpy="0 0 0"/>
   <parent link="base_link"/>
-  <child link="wheel_rf_1"/>
-  <axis xyz="-0.0 -1.0 0.0"/>
+  <child link="wheel_rf"/>
+  <axis xyz="0.0 1.0 0.0"/>
 </joint>
-<joint name="wheel_rb_1_joint" type="continuous">
-  <origin xyz="-0.11315 -0.142 0.03865" rpy="0 0 0"/>
+<joint name="wheel_rb_joint" type="continuous">
+  <origin xyz="-113.15e-03 -148.75e-03 0.0" rpy="0 0 0"/>
   <parent link="base_link"/>
-  <child link="wheel_rb_1"/>
-  <axis xyz="-0.0 -1.0 0.0"/>
+  <child link="wheel_rb"/>
+  <axis xyz="0.0 1.0 0.0"/>
 </joint>
 </robot>

Commit message: Retirada de Arquivos .STL Antigos e Adaptação ao Visual Simplificado

File: work_ws/src/salamander_bot/description/lidar.xacro (robot description, xacro)
@@ -8,7 +8,7 @@
   </inertial>
   <visual>
-    <origin xyz="-219.933902e-03 0.526156e-03 -29.599964e-03" rpy="0 0 0"/>
+    <origin xyz="0 0 0" rpy="0 0 0"/>
     <geometry>
-      <mesh filename="file://$(find salamander_bot)/meshes/rplidar_a1m8.stl" scale="0.001 0.001 0.001"/>
+      <cylinder length="0.0235" radius="0.035075" />
     </geometry>
     <material name="silver"/>

File: work_ws/src/salamander_bot/description/salamander_bot.xacro (robot description, xacro)
@@ -18,5 +18,5 @@
     <origin xyz="16.16414e-03 -4.12017e-03 -79.543971e-03" rpy="0 0 0"/>
     <geometry>
-      <mesh filename="package://salamander_bot/meshes/base_link.stl" scale="0.001 0.001 0.001"/>
+      <mesh filename="package://salamander_bot/meshes/base_link_collision.stl" scale="0.001 0.001 0.001"/>
     </geometry>
     <material name="silver"/>
@@ -36,9 +36,9 @@
   </inertial>
   <visual>
-    <origin xyz="-113.15e-03 -148.75e-03 -40.00e-03" rpy="0 0 0"/>
+    <origin xyz="0 0 0" rpy="${pi/2} 0 0"/>
     <geometry>
-      <mesh filename="package://salamander_bot/meshes/wheel_lf.stl" scale="0.001 0.001 0.001"/>
+      <cylinder length="0.0375" radius="0.04" />
     </geometry>
-    <material name="silver"/>
+    <material name="black"/>
   </visual>
   <collision>
@@ -56,9 +56,9 @@
   </inertial>
   <visual>
-    <origin xyz="113.15e-03 -148.75e-03 -40.00e-03" rpy="0 0 0"/>
+    <origin xyz="0 0 0" rpy="${pi/2} 0 0"/>
     <geometry>
-      <mesh filename="package://salamander_bot/meshes/wheel_lb.stl" scale="0.001 0.001 0.001"/>
+      <cylinder length="0.0375" radius="0.04" />
     </geometry>
-    <material name="silver"/>
+    <material name="black"/>
   </visual>
   <collision>
@@ -76,9 +76,9 @@
   </inertial>
   <visual>
-    <origin xyz="-113.15e-03 148.75e-03 -40.00e-03" rpy="0 0 0"/>
+    <origin xyz="0 0 0" rpy="${pi/2} 0 0"/>
     <geometry>
-      <mesh filename="package://salamander_bot/meshes/wheel_rf.stl" scale="0.001 0.001 0.001"/>
+      <cylinder length="0.0375" radius="0.04" />
     </geometry>
-    <material name="silver"/>
+    <material name="black"/>
   </visual>
   <collision>
@@ -96,9 +96,9 @@
   </inertial>
   <visual>
-    <origin xyz="113.15e-03 148.75e-03 -40.00e-03" rpy="0 0 0"/>
+    <origin xyz="0 0 0" rpy="${pi/2} 0 0"/>
     <geometry>
-      <mesh filename="package://salamander_bot/meshes/wheel_rb.stl" scale="0.001 0.001 0.001"/>
+      <cylinder length="0.0375" radius="0.04" />
     </geometry>
-    <material name="silver"/>
+    <material name="black"/>
   </visual>
   <collision>

Commit message: Adicionado Parâmetros de Inércia e Massa

File: work_ws/src/salamander_bot/description/lidar.xacro (robot description, xacro)
@@ -3,7 +3,7 @@
 <link name="rplidar_a1m8">
   <inertial>
-    <origin xyz="-0.016984302698711456 0.004773780112382523 0.02905054217183256" rpy="0 0 0"/>
-    <mass value="0.036021408390687064"/>
-    <inertia ixx="1.5e-05" iyy="1.2e-05" izz="2.3e-05" ixy="-0.0" iyz="0.0" ixz="-0.0"/>
+    <origin xyz="219.933902e-03 -0.526156e-03 29.599964e-03" rpy="0 0 0"/>
+    <mass value="125.885678e-03"/>
+    <inertia ixx="44511.257312e-09" iyy="44511.247312e-09" izz="77435.776975e-09" ixy="0.0" iyz="0.0" ixz="0.0"/>
   </inertial>
   <visual>

File: work_ws/src/salamander_bot/description/salamander_bot.xacro (robot description, xacro)
@@ -2,7 +2,5 @@
 <robot name="salamander_bot" xmlns:xacro="http://www.ros.org/wiki/xacro">
 <xacro:include filename="$(find salamander_bot)/description/colors.xacro" />
-<xacro:include filename="$(find salamander_bot)/description/arm_platform.xacro" />
 <xacro:include filename="$(find salamander_bot)/description/lidar.xacro" />
-<xacro:include filename="$(find salamander_bot)/description/webcam.xacro" />
 <xacro:include filename="$(find salamander_bot)/description/salamander_bot.ros2control" />
 <xacro:include filename="$(find salamander_bot)/description/salamander_bot.gazebo" />
@@ -11,7 +9,7 @@
 <link name="base_link">
   <inertial>
-    <origin xyz="-0.020630794834057973 0.00998649462328631 0.07392745780763998" rpy="0 0 0"/>
-    <mass value="4.267628583572636"/>
-    <inertia ixx="0.038378" iyy="0.079589" izz="0.097881" ixy="0.004056" iyz="-0.001772" ixz="0.008003"/>
+    <origin xyz="-26.696774e-03 5.87186e-03 79.358812e-03" rpy="0 0 0"/>
+    <mass value="4163.756809e-03"/>
+    <inertia ixx="0.03356" iyy="0.07829" izz="0.0953" ixy="0.003164" iyz="-0.0008321" ixz="0.007467"/>
   </inertial>
   <visual>
@@ -31,7 +29,7 @@
 <link name="wheel_lf">
   <inertial>
-    <origin xyz="6.732011406662686e-09 0.013415334217220576 -2.2496351934075953e-09" rpy="0 0 0"/>
-    <mass value="0.2163222450067834"/>
-    <inertia ixx="8.8e-05" iyy="0.00011" izz="8.8e-05" ixy="0.0" iyz="-0.0" ixz="0.0"/>
+    <origin xyz="113.15e-03 148.75e-03 40.0e-03" rpy="0 0 0"/>
+    <mass value="118.563707e-03"/>
+    <inertia ixx="61319.657896e-09" iyy="94850.959272e-09" izz="61319.670145e-09" ixy="0.0" iyz="0.0" ixz="0.0"/>
   </inertial>
   <visual>
@@ -51,7 +49,7 @@
 <link name="wheel_lb">
   <inertial>
-    <origin xyz="3.7014641768307044e-09 0.01344735270580652 -3.504848446189701e-09" rpy="0 0 0"/>
-    <mass value="0.21632224500656735"/>
-    <inertia ixx="8.8e-05" iyy="0.00011" izz="8.8e-05" ixy="-0.0" iyz="-0.0" ixz="0.0"/>
+    <origin xyz="-113.15e-03 148.75e-03 40.0e-03" rpy="0 0 0"/>
+    <mass value="118.563707e-03"/>
+    <inertia ixx="61319.657896e-09" iyy="94850.959272e-09" izz="61319.670145e-09" ixy="-0.0" iyz="0.0" ixz="0.0"/>
   </inertial>
   <visual>
@@ -71,7 +69,7 @@
 <link name="wheel_rf">
   <inertial>
-    <origin xyz="6.7541714166008404e-09 -0.013367918230393266 -2.072007607156756e-09" rpy="0 0 0"/>
-    <mass value="0.21632224116980406"/>
-    <inertia ixx="8.8e-05" iyy="0.00011" izz="8.8e-05" ixy="-0.0" iyz="0.0" ixz="0.0"/>
+    <origin xyz="113.15e-03 -148.75e-03 40.0e-03" rpy="0 0 0"/>
+    <mass value="118.563707e-03"/>
+    <inertia ixx="61319.657896e-09" iyy="94850.959272e-09" izz="61319.670145e-09" ixy="0.0" iyz="0.0" ixz="0.0"/>
   </inertial>
   <visual>
@@ -91,7 +89,7 @@
 <link name="wheel_rb">
   <inertial>
-    <origin xyz="3.723448854797695e-09 -0.013447353552784869 -3.327369837990979e-09" rpy="0 0 0"/>
-    <mass value="0.21632224116958718"/>
-    <inertia ixx="8.8e-05" iyy="0.00011" izz="8.8e-05" ixy="0.0" iyz="0.0" ixz="0.0"/>
+    <origin xyz="-113.15e-03 -148.75e-03 40.0e-03" rpy="0 0 0"/>
+    <mass value="118.563707e-03"/>
+    <inertia ixx="61319.657896e-09" iyy="94850.959272e-09" izz="61319.670145e-09" ixy="0.0" iyz="0.0" ixz="0.0"/>
   </inertial>
   <visual>
