Commit message: Correção nos Arquivos de URDF Provenientes de Erro no Merge

File: work_ws/src/salamander_bot/description/lidar.xacro (robot description, xacro)
@@ -1,16 +1,5 @@
 <?xml version="1.0"?>
 <robot name="salamander_bot" xmlns:xacro="http://www.ros.org/wiki/xacro">
-<<<<<<< HEAD
 <link name="rplidar_a1m8">
-=======
-<!-- Lidar joint -->
-<joint name="rplidar_a1m8_joint" type="fixed">
-  <origin xyz="0.236098 -0.004646 0.000956" rpy="0 0 0"/>
-  <parent link="base_link"/>
-  <child link="rplidar_a1m8_1"/>
-</joint>
-<!-- Lidar frame -->
-<link name="rplidar_a1m8_1">
->>>>>>> 473ca78 (Adicionado URDF Inicial de Robô Final (Manipulador + Chassi + Câmera + LIDAR) (Corrigir Câmera e LIDAR) & Correção na Modelagem da Cinemática Inversa da Movimentação - ESTAVA EM RAD/S AO INVÉS DE M/S :(((( (TESTAR))
   <inertial>
     <origin xyz="219.933902e-03 -0.526156e-03 29.599964e-03" rpy="0 0 0"/>
@@ -19,9 +8,5 @@
   </inertial>
   <visual>
-<<<<<<< HEAD
     <origin xyz="0 0 0" rpy="0 0 0"/>
-=======
-    <origin xyz="-0.236098 0.004646 -0.000956" rpy="0.0 0 0"/>
->>>>>>> 473ca78 (Adicionado URDF Inicial de Robô Final (Manipulador + Chassi + Câmera + LIDAR) (Corrigir Câmera e LIDAR) & Correção na Modelagem da Cinemática Inversa da Movimentação - ESTAVA EM RAD/S AO INVÉS DE M/S :(((( (TESTAR))
     <geometry>
       <cylinder length="0.0235" radius="0.035075" />
@@ -30,9 +15,5 @@
   </visual>
   <collision>
-<<<<<<< HEAD
     <origin xyz="0 0 0" rpy="0 0 0"/>
-=======
-    <origin xyz="-0.236098 0.004646 -0.000956" rpy="0.0 0 0"/>
->>>>>>> 473ca78 (Adicionado URDF Inicial de Robô Final (Manipulador + Chassi + Câmera + LIDAR) (Corrigir Câmera e LIDAR) & Correção na Modelagem da Cinemática Inversa da Movimentação - ESTAVA EM RAD/S AO INVÉS DE M/S :(((( (TESTAR))
     <geometry>
       <cylinder length="0.0235" radius="0.035075" />

File: work_ws/src/salamander_bot/description/salamander_bot.xacro (robot description, xacro)
@@ -2,7 +2,5 @@
 <robot name="salamander_bot" xmlns:xacro="http://www.ros.org/wiki/xacro">
 <xacro:include filename="$(find salamander_bot)/description/colors.xacro" />
-<xacro:include filename="$(find salamander_bot)/description/arm_platform.xacro" />
 <xacro:include filename="$(find salamander_bot)/description/lidar.xacro" />
-<xacro:include filename="$(find salamander_bot)/description/webcam.xacro" />
 <xacro:include filename="$(find salamander_bot)/description/salamander_bot.ros2control" />
 <xacro:include filename="$(find salamander_bot)/description/salamander_bot.gazebo" />

Commit message: Corrigindo URDF do robo

File: work_ws/src/salamander_bot/description/lidar.xacro (robot description, xacro)
@@ -1,5 +1,5 @@
 <?xml version="1.0"?>
 <robot name="salamander_bot" xmlns:xacro="http://www.ros.org/wiki/xacro">
-<link name="rplidar_a1m8">
+<link name="rplidar_a1m8_1">
   <inertial>
     <origin xyz="219.933902e-03 -0.526156e-03 29.599964e-03" rpy="0 0 0"/>
@@ -8,5 +8,5 @@
   </inertial>
   <visual>
-    <origin xyz="0 0 0" rpy="0 0 0"/>
+    <origin xyz="0 0 0.04" rpy="0 0 0"/>
     <geometry>
       <cylinder length="0.0235" radius="0.035075" />
@@ -15,5 +15,5 @@
   </visual>
   <collision>
-    <origin xyz="0 0 0" rpy="0 0 0"/>
+    <origin xyz="0 0 0.04" rpy="0 0 0"/>
     <geometry>
       <cylinder length="0.0235" radius="0.035075" />
@@ -21,7 +21,7 @@
   </collision>
 </link>
-<joint name="rplidar_a1m8_joint" type="fixed">
+<joint name="rplidar_a1m8_1_joint" type="fixed">
   <parent link="base_link"/>
-  <child link="rplidar_a1m8"/>
+  <child link="rplidar_a1m8_1"/>
   <origin xyz="219.933902e-03 -0.526156e-03 -10.400036e-03" rpy="0 0 0"/>
 </joint>

File: work_ws/src/salamander_bot/description/salamander_bot.xacro (robot description, xacro)
@@ -14,5 +14,5 @@
   </inertial>
   <visual>
-    <origin xyz="16.16414e-03 -4.12017e-03 -79.543971e-03" rpy="0 0 0"/>
+    <origin xyz="16.16414e-03 -4.12017e-03 -39.543971e-03" rpy="0 0 0"/>
     <geometry>
       <mesh filename="package://salamander_bot/meshes/base_link_collision.stl" scale="0.001 0.001 0.001"/>
@@ -21,5 +21,5 @@
   </visual>
   <collision>
-    <origin xyz="16.16414e-03 -4.12017e-03 -79.543971e-03" rpy="0 0 0"/>
+    <origin xyz="16.16414e-03 -4.12017e-03 -39.543971e-03" rpy="0 0 0"/>
     <geometry>
       <mesh filename="package://salamander_bot/meshes/base_link_collision.stl" scale="0.001 0.001 0.001"/>
@@ -27,5 +27,5 @@
   </collision>
 </link>
-<link name="wheel_lf">
+<link name="wheel_lf_1">
   <inertial>
     <origin xyz="113.15e-03 148.75e-03 40.0e-03" rpy="0 0 0"/>
@@ -34,5 +34,5 @@
   </inertial>
   <visual>
-    <origin xyz="0 0 0" rpy="${pi/2} 0 0"/>
+    <origin xyz="0 0 0.04" rpy="${pi/2} 0 0"/>
     <geometry>
       <cylinder length="0.0375" radius="0.04" />
@@ -41,5 +41,5 @@
   </visual>
   <collision>
-    <origin xyz="0 0 0" rpy="${pi/2} 0 0"/>
+    <origin xyz="0 0 0.04" rpy="${pi/2} 0 0"/>
     <geometry>
       <cylinder length="0.0375" radius="0.04" />
@@ -47,5 +47,5 @@
   </collision>
 </link>
-<link name="wheel_lb">
+<link name="wheel_lb_1">
   <inertial>
     <origin xyz="-113.15e-03 148.75e-03 40.0e-03" rpy="0 0 0"/>
@@ -54,5 +54,5 @@
   </inertial>
   <visual>
-    <origin xyz="0 0 0" rpy="${pi/2} 0 0"/>
+    <origin xyz="0 0 0.04" rpy="${pi/2} 0 0"/>
     <geometry>
       <cylinder length="0.0375" radius="0.04" />
@@ -61,5 +61,5 @@
   </visual>
   <collision>
-    <origin xyz="0 0 0" rpy="${pi/2} 0 0"/>
+    <origin xyz="0 0 0.04" rpy="${pi/2} 0 0"/>
     <geometry>
       <cylinder length="0.0375" radius="0.04" />
@@ -67,5 +67,5 @@
   </collision>
 </link>
-<link name="wheel_rf">
+<link name="wheel_rf_1">
   <inertial>
     <origin xyz="113.15e-03 -148.75e-03 40.0e-03" rpy="0 0 0"/>
@@ -74,5 +74,5 @@
   </inertial>
   <visual>
-    <origin xyz="0 0 0" rpy="${pi/2} 0 0"/>
+    <origin xyz="0 0 0.04" rpy="${pi/2} 0 0"/>
     <geometry>
       <cylinder length="0.0375" radius="0.04" />
@@ -81,5 +81,5 @@
   </visual>
   <collision>
-    <origin xyz="0 0 0" rpy="${pi/2} 0 0"/>
+    <origin xyz="0 0 0.04" rpy="${pi/2} 0 0"/>
     <geometry>
       <cylinder length="0.0375" radius="0.04" />
@@ -87,5 +87,5 @@
   </collision>
 </link>
-<link name="wheel_rb">
+<link name="wheel_rb_1">
   <inertial>
     <origin xyz="-113.15e-03 -148.75e-03 40.0e-03" rpy="0 0 0"/>
@@ -94,5 +94,5 @@
   </inertial>
   <visual>
-    <origin xyz="0 0 0" rpy="${pi/2} 0 0"/>
+    <origin xyz="0 0 0.04" rpy="${pi/2} 0 0"/>
     <geometry>
       <cylinder length="0.0375" radius="0.04" />
@@ -101,5 +101,5 @@
   </visual>
   <collision>
-    <origin xyz="0 0 0" rpy="${pi/2} 0 0"/>
+    <origin xyz="0 0 0.04" rpy="${pi/2} 0 0"/>
     <geometry>
       <cylinder length="0.0375" radius="0.04" />
@@ -112,26 +112,26 @@
   <origin xyz="0.0 0.0 40.0e-03" rpy="0.0 0.0 0.0"/>
 </joint>
-<joint name="wheel_lf_joint" type="continuous">
+<joint name="wheel_lf_1_joint" type="continuous">
   <origin xyz="113.15e-03 148.75e-03 0.0" rpy="0 0 0"/>
   <parent link="base_link"/>
-  <child link="wheel_lf"/>
+  <child link="wheel_lf_1"/>
   <axis xyz="0.0 1.0 0.0"/>
 </joint>
-<joint name="wheel_lb_joint" type="continuous">
+<joint name="wheel_lb_1_joint" type="continuous">
   <origin xyz="-113.15e-03 148.75e-03 0.0" rpy="0 0 0"/>
   <parent link="base_link"/>
-  <child link="wheel_lb"/>
+  <child link="wheel_lb_1"/>
   <axis xyz="0.0 1.0 0.0"/>
 </joint>
-<joint name="wheel_rf_joint" type="continuous">
+<joint name="wheel_rf_1_joint" type="continuous">
   <origin xyz="113.15e-03 -148.75e-03 0.0" rpy="0 0 0"/>
   <parent link="base_link"/>
-  <child link="wheel_rf"/>
+  <child link="wheel_rf_1"/>
   <axis xyz="0.0 1.0 0.0"/>
 </joint>
-<joint name="wheel_rb_joint" type="continuous">
+<joint name="wheel_rb_1_joint" type="continuous">
   <origin xyz="-113.15e-03 -148.75e-03 0.0" rpy="0 0 0"/>
   <parent link="base_link"/>
-  <child link="wheel_rb"/>
+  <child link="wheel_rb_1"/>
   <axis xyz="0.0 1.0 0.0"/>
 </joint>

Commit message: Ajuste de erro URDF

File: work_ws/src/salamander_bot/description/lidar.xacro (robot description, xacro)
@@ -3,5 +3,5 @@
 <link name="rplidar_a1m8_1">
   <inertial>
-    <origin xyz="219.933902e-03 -0.526156e-03 29.599964e-03" rpy="0 0 0"/>
+    <origin xyz="-0.526156e-03 219.933902e-03 29.599964e-03" rpy="0 0 0"/>
     <mass value="125.885678e-03"/>
     <inertia ixx="44511.257312e-09" iyy="44511.247312e-09" izz="77435.776975e-09" ixy="0.0" iyz="0.0" ixz="0.0"/>
@@ -24,5 +24,6 @@
   <parent link="base_link"/>
   <child link="rplidar_a1m8_1"/>
-  <origin xyz="219.933902e-03 -0.526156e-03 -10.400036e-03" rpy="0 0 0"/>
+  <!-- X e Y invertidos para o sensor não flutuar do lado do robô -->
+  <origin xyz="-0.526156e-03 219.933902e-03 -10.400036e-03" rpy="0 0 0"/>
 </joint>
 </robot>

File: work_ws/src/salamander_bot/description/salamander_bot.xacro (robot description, xacro)
@@ -113,5 +113,5 @@
 </joint>
 <joint name="wheel_lf_1_joint" type="continuous">
-  <origin xyz="113.15e-03 148.75e-03 0.0" rpy="0 0 0"/>
+  <origin xyz="148.75e-03 113.15e-03 0.0" rpy="0 0 0"/>
   <parent link="base_link"/>
   <child link="wheel_lf_1"/>
@@ -119,5 +119,5 @@
 </joint>
 <joint name="wheel_lb_1_joint" type="continuous">
-  <origin xyz="-113.15e-03 148.75e-03 0.0" rpy="0 0 0"/>
+  <origin xyz="148.75e-03 -113.15e-03 0.0" rpy="0 0 0"/>
   <parent link="base_link"/>
   <child link="wheel_lb_1"/>
@@ -125,5 +125,5 @@
 </joint>
 <joint name="wheel_rf_1_joint" type="continuous">
-  <origin xyz="113.15e-03 -148.75e-03 0.0" rpy="0 0 0"/>
+  <origin xyz="-148.75e-03 113.15e-03 0.0" rpy="0 0 0"/>
   <parent link="base_link"/>
   <child link="wheel_rf_1"/>
@@ -131,5 +131,5 @@
 </joint>
 <joint name="wheel_rb_1_joint" type="continuous">
-  <origin xyz="-113.15e-03 -148.75e-03 0.0" rpy="0 0 0"/>
+  <origin xyz="-148.75e-03 -113.15e-03 0.0" rpy="0 0 0"/>
   <parent link="base_link"/>
   <child link="wheel_rb_1"/>

Commit message: Teste de Orientação de Coordenadas

File: work_ws/src/salamander_bot/description/lidar.xacro (robot description, xacro)
@@ -3,10 +3,10 @@
 <link name="rplidar_a1m8_1">
   <inertial>
-    <origin xyz="-0.526156e-03 219.933902e-03 29.599964e-03" rpy="0 0 0"/>
+    <origin xyz="219.933902e-03 -0.526156e-03 29.599964e-03" rpy="0 0 0"/>
     <mass value="125.885678e-03"/>
     <inertia ixx="44511.257312e-09" iyy="44511.247312e-09" izz="77435.776975e-09" ixy="0.0" iyz="0.0" ixz="0.0"/>
   </inertial>
   <visual>
-    <origin xyz="0 0 0.04" rpy="0 0 0"/>
+    <origin xyz="0 0 0" rpy="0 0 0"/>
     <geometry>
       <cylinder length="0.0235" radius="0.035075" />
@@ -15,5 +15,5 @@
   </visual>
   <collision>
-    <origin xyz="0 0 0.04" rpy="0 0 0"/>
+    <origin xyz="0 0 0" rpy="0 0 0"/>
     <geometry>
       <cylinder length="0.0235" radius="0.035075" />
@@ -24,6 +24,5 @@
   <parent link="base_link"/>
   <child link="rplidar_a1m8_1"/>
-  <!-- X e Y invertidos para o sensor não flutuar do lado do robô -->
-  <origin xyz="-0.526156e-03 219.933902e-03 -10.400036e-03" rpy="0 0 0"/>
+  <origin xyz="219.933902e-03 -0.526156e-03 -10.400036e-03" rpy="0 0 0"/>
 </joint>
 </robot>

File: work_ws/src/salamander_bot/description/salamander_bot.xacro (robot description, xacro)
@@ -14,5 +14,5 @@
   </inertial>
   <visual>
-    <origin xyz="16.16414e-03 -4.12017e-03 -39.543971e-03" rpy="0 0 ${pi/2}"/>
+    <origin xyz="16.16414e-03 -4.12017e-03 -79.543971e-03" rpy="0 0 0"/>
     <geometry>
       <mesh filename="package://salamander_bot/meshes/base_link_collision.stl" scale="0.001 0.001 0.001"/>
@@ -21,5 +21,5 @@
   </visual>
   <collision>
-    <origin xyz="16.16414e-03 -4.12017e-03 -39.543971e-03" rpy="0 0 ${pi/2}"/>
+    <origin xyz="16.16414e-03 -4.12017e-03 -79.543971e-03" rpy="0 0 0"/>
     <geometry>
       <mesh filename="package://salamander_bot/meshes/base_link_collision.stl" scale="0.001 0.001 0.001"/>
@@ -34,5 +34,5 @@
   </inertial>
   <visual>
-    <origin xyz="0 0 0.04" rpy="${pi/2} 0 0"/>
+    <origin xyz="0 0 0" rpy="${pi/2} 0 0"/>
     <geometry>
       <cylinder length="0.0375" radius="0.04" />
@@ -41,5 +41,5 @@
   </visual>
   <collision>
-    <origin xyz="0 0 0.04" rpy="${pi/2} 0 0"/>
+    <origin xyz="0 0 0" rpy="${pi/2} 0 0"/>
     <geometry>
       <cylinder length="0.0375" radius="0.04" />
@@ -54,5 +54,5 @@
   </inertial>
   <visual>
-    <origin xyz="0 0 0.04" rpy="${pi/2} 0 0"/>
+    <origin xyz="0 0 0" rpy="${pi/2} 0 0"/>
     <geometry>
       <cylinder length="0.0375" radius="0.04" />
@@ -61,5 +61,5 @@
   </visual>
   <collision>
-    <origin xyz="0 0 0.04" rpy="${pi/2} 0 0"/>
+    <origin xyz="0 0 0" rpy="${pi/2} 0 0"/>
     <geometry>
       <cylinder length="0.0375" radius="0.04" />
@@ -74,5 +74,5 @@
   </inertial>
   <visual>
-    <origin xyz="0 0 0.04" rpy="${pi/2} 0 0"/>
+    <origin xyz="0 0 0" rpy="${pi/2} 0 0"/>
     <geometry>
       <cylinder length="0.0375" radius="0.04" />
@@ -81,5 +81,5 @@
   </visual>
   <collision>
-    <origin xyz="0 0 0.04" rpy="${pi/2} 0 0"/>
+    <origin xyz="0 0 0" rpy="${pi/2} 0 0"/>
     <geometry>
       <cylinder length="0.0375" radius="0.04" />
@@ -94,5 +94,5 @@
   </inertial>
   <visual>
-    <origin xyz="0 0 0.04" rpy="${pi/2} 0 0"/>
+    <origin xyz="0 0 0" rpy="${pi/2} 0 0"/>
     <geometry>
       <cylinder length="0.0375" radius="0.04" />
@@ -101,5 +101,5 @@
   </visual>
   <collision>
-    <origin xyz="0 0 0.04" rpy="${pi/2} 0 0"/>
+    <origin xyz="0 0 0" rpy="${pi/2} 0 0"/>
     <geometry>
       <cylinder length="0.0375" radius="0.04" />
@@ -113,5 +113,5 @@
 </joint>
 <joint name="wheel_lf_1_joint" type="continuous">
-  <origin xyz="148.75e-03 113.15e-03 0.0" rpy="0 0 0"/>
+  <origin xyz="113.15e-03 148.75e-03 0.0" rpy="0 0 0"/>
   <parent link="base_link"/>
   <child link="wheel_lf_1"/>
@@ -119,5 +119,5 @@
 </joint>
 <joint name="wheel_lb_1_joint" type="continuous">
-  <origin xyz="148.75e-03 -113.15e-03 0.0" rpy="0 0 0"/>
+  <origin xyz="-113.15e-03 148.75e-03 0.0" rpy="0 0 0"/>
   <parent link="base_link"/>
   <child link="wheel_lb_1"/>
@@ -125,5 +125,5 @@
 </joint>
 <joint name="wheel_rf_1_joint" type="continuous">
-  <origin xyz="-148.75e-03 113.15e-03 0.0" rpy="0 0 0"/>
+  <origin xyz="113.15e-03 -148.75e-03 0.0" rpy="0 0 0"/>
   <parent link="base_link"/>
   <child link="wheel_rf_1"/>
@@ -131,5 +131,5 @@
 </joint>
 <joint name="wheel_rb_1_joint" type="continuous">
-  <origin xyz="-148.75e-03 -113.15e-03 0.0" rpy="0 0 0"/>
+  <origin xyz="-113.15e-03 -148.75e-03 0.0" rpy="0 0 0"/>
   <parent link="base_link"/>
   <child link="wheel_rb_1"/>
