Commit message: URDF Câmera + Braço (Ajustar Inércia e Centro de Massa Para Simulação)

File: work_ws/src/salamander_bot/description/arm_platform.xacro (robot description, xacro)
@@ -111,10 +111,16 @@
   <child link="height_link"/>
   <axis xyz="0.0 0.0 1.0"/>
+  <limit effort="25" velocity="0.05"/>
 </joint>
-<joint name="arm_joint" type="continuous">
+<joint name="arm_joint" type="revolute">
   <origin xyz="-0.045e-03 -43.666664e-03 162.505e-03" rpy="0 0 0"/>
   <parent link="height_link"/>
   <child link="arm_link"/>
   <axis xyz="0.0 1.0 0.0"/>
+  <limit
+    lower="${-pi/6}"
+    upper="${5*pi/18}"
+    effort="25"
+    velocity="0.05"/>
 </joint>
 <joint name="gripper_left_joint" type="prismatic">

File: work_ws/src/salamander_bot/description/lidar.xacro (robot description, xacro)
@@ -3,5 +3,5 @@
 <!-- Lidar joint: Mantém a matemática correta para o Nav2 -->
 <joint name="rplidar_a1m8_joint" type="fixed">
-  <origin xyz="0.236098 -0.004646 0.000956" rpy="3.14159 0 1.5708"/>
+  <origin xyz="0.236098 -0.004646 0.000956" rpy="${pi} 0 ${pi/2}"/>
   <parent link="base_link"/>
   <child link="rplidar_a1m8_1"/>
@@ -16,5 +16,5 @@
   <visual>
     <!-- A mágica matemática: isso anula a junta para o desenho renderizar como no CAD -->
-    <origin xyz="0.004646 -0.236098 0.000956" rpy="3.14159 0 1.5708"/>
+    <origin xyz="0.004646 -0.236098 0.000956" rpy="${pi} 0 ${pi/2}"/>
     <geometry>
       <mesh filename="package://salamander_bot/meshes/rplidar_a1m8_1.stl" scale="0.001 0.001 0.001"/>
@@ -24,5 +24,5 @@
   <collision>
     <!-- A mágica matemática também na colisão -->
-    <origin xyz="0.004646 -0.236098 0.000956" rpy="3.14159 0 1.5708"/>
+    <origin xyz="0.004646 -0.236098 0.000956" rpy="${pi} 0 ${pi/2}"/>
     <geometry>
       <mesh filename="package://salamander_bot/meshes/rplidar_a1m8_1.stl" scale="0.001 0.001 0.001"/>

File: work_ws/src/salamander_bot/description/salamander_bot.xacro (robot description, xacro)
@@ -3,4 +3,6 @@
 <xacro:include filename="$(find salamander_bot)/description/colors.xacro" />
 <xacro:include filename="$(find salamander_bot)/description/lidar.xacro" />
+<xacro:include filename="$(find salamander_bot)/description/webcam.xacro" />
+<xacro:include filename="$(find salamander_bot)/description/arm_platform.xacro" />
 <xacro:include filename="$(find salamander_bot)/description/salamander_bot.ros2control" />
 <xacro:include filename="$(find salamander_bot)/description/salamander_bot.gazebo" />

File: work_ws/src/salamander_bot/description/webcam.xacro (robot description, xacro)
@@ -1,5 +1,5 @@
 <?xml version="1.0"?>
 <robot name="salamander_bot" xmlns:xacro="http://www.ros.org/wiki/xacro">
-<link name="webcam">
+<link name="webcam_link">
   <inertial>
     <origin xyz="18.314038e-03 46.775002e-03 177.993585e-03" rpy="0 0 0"/>
@@ -8,5 +8,5 @@
   </inertial>
   <visual>
-    <origin xyz="-12.753605e-03 0.16967e-03 51.105768e-03" rpy="0 0 0"/>
+    <origin xyz="-50.753605e-03 -12.16967e-03 0.105768e-03" rpy="${pi/2} 0 ${pi/2}"/>
     <geometry>
       <mesh filename="package://salamander_bot/meshes/webcam.stl" scale="0.001 0.001 0.001"/>
@@ -15,5 +15,5 @@
   </visual>
   <collision>
-    <origin xyz="-12.753605e-03 0.16967e-03 51.105768e-03" rpy="0 0 0"/>
+    <origin xyz="-50.753605e-03 -12.16967e-03 0.105768e-03" rpy="${pi/2} 0 ${pi/2}"/>
     <geometry>
       <mesh filename="package://salamander_bot/meshes/webcam.stl" scale="0.001 0.001 0.001"/>
@@ -24,5 +24,11 @@
   <origin xyz="0.504998e-03 42.70432e-03 188.254995e-03" rpy="0 0 0"/>
   <parent link="height_link"/>
-  <child link="webcam"/>
+  <child link="webcam_link"/>
+</joint>
+<link name="webcam_link_optical"></link>
+<joint name="webcam_optical_joint" type="fixed">
+  <origin xyz="40e-03 -10e-03 -15e-03" rpy="${-pi/2} 0 ${-pi/2}"/>
+  <parent link="webcam_link"/>
+  <child link="webcam_link_optical"/>
 </joint>
 </robot>

Commit message: Testando com um frame fixo na base do manipulador

File: work_ws/src/salamander_bot/description/arm_platform.xacro (robot description, xacro)
@@ -21,4 +21,12 @@
   </collision>
 </link>
+<link name="arm_base_static">
+</link>
+<joint name="arm_base_static_joint" type="fixed">
+  <!-- Mesma origem do height_joint -->
+  <origin xyz="-106.224243e-03 -4.427118e-03 21.00e-03" rpy="0 0 0"/>
+  <parent link="platform_link"/>
+  <child link="arm_base_static"/>
+</joint>
 <link name="height_link">
   <inertial>
