Commit message: Arrumando o erro da navegação

File: work_ws/install/salamander_bot/share/salamander_bot/description/colors.xacro (robot description, xacro)
@@ -1 +1,18 @@
-/home/enzo/droid/WORK-2026/work_ws/src/salamander_bot/description/colors.xacro
+<?xml version="1.0"?>
+<robot xmlns:xacro="http://www.ros.org/wiki/xacro">
+    <material name="white">
+        <color rgba="1.0 1.0 1.0 1.0"/>
+    </material>
+    <material name="orange">
+        <color rgba="1.0 0.3 0.1 1.0"/>
+    </material>
+    <material name="blue">
+        <color rgba="0.2 0.2 1.0 1.0"/>
+    </material>
+    <material name="black">
+        <color rgba="0.0 0.0 0.0 1.0"/>
+    </material>
+    <material name="silver">
+        <color rgba="0.7 0.7 0.7 1.0"/>
+    </material>
+</robot>

File: work_ws/install/salamander_bot/share/salamander_bot/description/lidar.xacro (robot description, xacro)
@@ -1 +1,54 @@
-/home/enzo/droid/WORK-2026/work_ws/src/salamander_bot/description/lidar.xacro
+<?xml version="1.0"?>
+<robot name="salamander_bot" xmlns:xacro="http://www.ros.org/wiki/xacro">
+<!-- Lidar joint -->
+<joint name="Rigid 11" type="fixed">
+  <origin xyz="0.236098 -0.004646 0.000956" rpy="0 0 0"/>
+  <parent link="base_link"/>
+  <child link="rplidar_a1m8_1"/>
+</joint>
+<!-- Lidar frame -->
+<link name="rplidar_a1m8_1">
+  <inertial>
+    <origin xyz="-0.016984302698711456 0.004773780112382523 0.02905054217183256" rpy="0 0 0"/>
+    <mass value="0.036021408390687064"/>
+    <inertia ixx="1.5e-05" iyy="1.2e-05" izz="2.3e-05" ixy="-0.0" iyz="0.0" ixz="-0.0"/>
+  </inertial>
+  <visual>
+    <origin xyz="-0.236098 0.004646 -0.000956" rpy="0 0 0"/>
+    <geometry>
+      <mesh filename="file://$(find salamander_bot)/meshes/rplidar_a1m8_1.stl" scale="0.001 0.001 0.001"/>
+    </geometry>
+    <material name="silver"/>
+  </visual>
+  <collision>
+    <origin xyz="-0.236098 0.004646 -0.000956" rpy="0 0 0"/>
+    <geometry>
+      <mesh filename="file://$(find salamander_bot)/meshes/rplidar_a1m8_1.stl" scale="0.001 0.001 0.001"/>
+    </geometry>
+  </collision>
+</link>
+<gazebo reference="rplidar_a1m8_1">
+  <sensor name="lidar" type="lidar">
+    <pose>0 0 0 0 0 0</pose>
+    <update_rate>10</update_rate>
+    <visualize>false</visualize>
+    <topic>/sim/scan</topic>
+    <lidar>
+      <scan>
+        <horizontal>
+          <samples>360</samples>
+          <resolution>1</resolution>
+          <min_angle>-3.14</min_angle>
+          <max_angle>3.14</max_angle>
+        </horizontal>
+      </scan>
+      <range>
+        <min>0.15</min>
+        <max>12.0</max>
+      </range>
+    </lidar>
+    <gz_frame_id>rplidar_a1m8_1</gz_frame_id>
+    <always_on>true</always_on>
+  </sensor>
+</gazebo>
+</robot>

File: work_ws/install/salamander_bot/share/salamander_bot/description/robot.urdf.xacro (robot description, xacro)
@@ -1 +1,7 @@
-/home/enzo/droid/WORK-2026/work_ws/src/salamander_bot/description/robot.urdf.xacro
+<?xml version="1.0"?>
+<robot name="salamander_bot" xmlns:xacro="http://www.ros.org/wiki/xacro">
+    <!-- Robot Core File -->
+    <xacro:include filename="robot_core.xacro" />
+    <!-- Lidar -->
+    <xacro:include filename="lidar.xacro" />
+</robot>

File: work_ws/install/salamander_bot/share/salamander_bot/description/robot_core.xacro (robot description, xacro)
@@ -1 +1,145 @@
-/home/enzo/droid/WORK-2026/work_ws/src/salamander_bot/description/robot_core.xacro
+<?xml version="1.0" ?>
+<robot xmlns:xacro="http://www.ros.org/wiki/xacro">
+<xacro:include filename="$(find salamander_bot)/description/colors.xacro" />
+<xacro:include filename="$(find salamander_bot)/description/salamander_bot.ros2control" />
+<xacro:include filename="$(find salamander_bot)/description/salamander_bot.gazebo" />
+<!-- Adicionado SLAM -->
+<link name="base_link">
+</link>
+<joint name="base_footprint_joint" type="fixed">
+  <parent link="base_link"/>
+  <child link="base_footprint"/>
+  <origin xyz="0.0 0.0 0.0" rpy="0.0 0.0 0.0"/>
+</joint>
+<link name="base_footprint">
+</link>
+<!-- fim SLAM -->
+<link name="chassis">
+  <inertial>
+    <origin xyz="-0.031027251343893784 0.006588573186617724 0.08110908537527221" rpy="0 0 0"/>
+    <mass value="4.3632165889636445"/>
+    <inertia ixx="0.042227" iyy="0.075384" izz="0.090994" ixy="0.004338" iyz="-0.000531" ixz="0.008602"/>
+  </inertial>
+  <visual>
+    <origin xyz="0 0 0" rpy="0 0 0"/>
+    <geometry>
+      <mesh filename="file://$(find salamander_bot)/meshes/base_link.stl" scale="0.001 0.001 0.001"/>
+    </geometry>
+    <material name="silver"/>
+  </visual>
+  <collision>
+    <origin xyz="0 0 0" rpy="0 0 0"/>
+    <geometry>
+      <mesh filename="file://$(find salamander_bot)/meshes/base_link.stl" scale="0.001 0.001 0.001"/>
+    </geometry>
+  </collision>
+</link>
+<joint name="chassis_joint" type="fixed">
+  <parent link="base_link"/>
+  <child link="chassis"/>
+  <origin xyz="0.0 0.0 0.0"/>
+</joint>
+<link name="wheel_lf_1">
+  <inertial>
+    <origin xyz="0.11315 0.142 -0.03865" rpy="0 0 0"/>
+    <mass value="0.216322"/>
+    <inertia ixx="8.8e-05" iyy="0.00011" izz="8.8e-05" ixy="0.0" iyz="0.0" ixz="0.0"/>
+  </inertial>
+  <visual>
+    <origin xyz="0 0 0" rpy="0 0 0"/>
+    <geometry>
+      <mesh filename="file://$(find salamander_bot)/meshes/wheel_lf_1.stl" scale="0.001 0.001 0.001"/>
+    </geometry>
+    <material name="black"/>
+  </visual>
+  <collision>
+    <origin xyz="0 0 0" rpy="0 0 0"/>
+    <geometry>
+      <mesh filename="file://$(find salamander_bot)/meshes/wheel_lf_1.stl" scale="0.001 0.001 0.001"/>
+    </geometry>
+  </collision>
+</link>
+<joint name="wheel_lf_joint" type="continuous">
+  <origin xyz="0.0 0.0 0.0" rpy="0 0 0"/> <parent link="base_link"/>
+  <child link="wheel_lf_1"/>
+  <axis xyz="0.0 1.0 0.0"/>
+</joint>
+<link name="wheel_lb_1">
+  <inertial>
+    <origin xyz="-0.11315 0.142 -0.03865" rpy="0 0 0"/>
+    <mass value="0.216322"/>
+    <inertia ixx="8.8e-05" iyy="0.00011" izz="8.8e-05" ixy="0.0" iyz="0.0" ixz="0.0"/>
+  </inertial>
+  <visual>
+    <origin xyz="0 0 0" rpy="0 0 0"/>
+    <geometry>
+      <mesh filename="file://$(find salamander_bot)/meshes/wheel_lb_1.stl" scale="0.001 0.001 0.001"/>
+    </geometry>
+    <material name="black"/>
+  </visual>
+  <collision>
+    <origin xyz="0 0 0" rpy="0 0 0"/>
+    <geometry>
+      <mesh filename="file://$(find salamander_bot)/meshes/wheel_lb_1.stl" scale="0.001 0.001 0.001"/>
+    </geometry>
+  </collision>
+</link>
+<joint name="wheel_lb_joint" type="continuous">
+  <origin xyz="0.0 0.0 0.0" rpy="0 0 0"/>
+  <parent link="base_link"/>
+  <child link="wheel_lb_1"/>
+  <axis xyz="0.0 1.0 0.0"/>
+</joint>
+<link name="wheel_rf_1">
+  <inertial>
+    <origin xyz="0.11315 -0.142 -0.03865" rpy="0 0 0"/>
+    <mass value="0.216322"/>
+    <inertia ixx="8.8e-05" iyy="0.00011" izz="8.8e-05" ixy="0.0" iyz="0.0" ixz="0.0"/>
+  </inertial>
+  <visual>
+    <origin xyz="0 0 0" rpy="0 0 0"/>
+    <geometry>
+      <mesh filename="file://$(find salamander_bot)/meshes/wheel_rf_1.stl" scale="0.001 0.001 0.001"/>
+    </geometry>
+    <material name="black"/>
+  </visual>
+  <collision>
+    <origin xyz="0 0 0" rpy="0 0 0"/>
+    <geometry>
+      <mesh filename="file://$(find salamander_bot)/meshes/wheel_rf_1.stl" scale="0.001 0.001 0.001"/>
+    </geometry>
+  </collision>
+</link>
+<joint name="wheel_rf_joint" type="continuous">
+  <origin xyz="0.0 0.0 0.0" rpy="0 0 0"/>
+  <parent link="base_link"/>
+  <child link="wheel_rf_1"/>
+  <axis xyz="0.0 1.0 0.0"/>
+</joint>
+<link name="wheel_rb_1">
+  <inertial>
+    <origin xyz="-0.11315 -0.142 -0.03865" rpy="0 0 0"/>
+    <mass value="0.216322"/>
+    <inertia ixx="8.8e-05" iyy="0.00011" izz="8.8e-05" ixy="0.0" iyz="0.0" ixz="0.0"/>
+  </inertial>
+  <visual>
+    <origin xyz="0 0 0" rpy="0 0 0"/>
+    <geometry>
+      <mesh filename="file://$(find salamander_bot)/meshes/wheel_rb_1.stl" scale="0.001 0.001 0.001"/>
+    </geometry>
+    <material name="black"/>
+  </visual>
+  <collision>
+    <origin xyz="0 0 0" rpy="0 0 0"/>
+    <geometry>
+      <mesh filename="file://$(find salamander_bot)/meshes/wheel_rb_1.stl" scale="0.001 0.001 0.001"/>
+    </geometry>
+  </collision>
+</link>
+<joint name="wheel_rb_joint" type="continuous">
+  <origin xyz="0.0 0.0 0.0" rpy="0 0 0"/>
+  <parent link="base_link"/>
+  <child link="wheel_rb_1"/>
+  <axis xyz="0.0 1.0 0.0"/>
+</joint>
+</robot>
